File: cortex-face-1.sch (KiCad schematic (older format))
At the start: 170 parts

Commit message: PCB started
Footprints defined
Parts:
- D1, D10, D11, D12, D13, D14, D15, D16, D17, D18, D19, D2, D20, D21, D22, D23, D24, D25, D26, D27, D28, D29, D3, D30, D31, D32, D33, D34, D35, D36, D37, D38, D39, D4, D40, D41, D42, D43, D44, D45, D46, D47, D48, D49, D5, D50, D51, D52, D53, D54, D55, D56, D57, D58, D59, D6, D60, D61, D62, D63, D64, D65, D66, D67, D68, D69, D7, D70, D71, D72, D73, D74, D75, D76, D77, D78, D79, D8, D80, D81, D82, D83, D9: renamed from D?; footprint (none) -> Keebio-Parts:Diode
- J1: renamed from J?; footprint (none) -> Connector_Wire:SolderWirePad_1x04_P3.81mm_Drill1mm
- MX_'"1: renamed from MX_'"; footprint (none) -> MX_Alps_Hybrid:MX-1U-NoLED
- MX_,<1: renamed from MX_,<; footprint (none) -> MX_Alps_Hybrid:MX-1U-NoLED
- MX_-_1: renamed from MX_-_; footprint (none) -> MX_Alps_Hybrid:MX-1U-NoLED
- MX_.>1: renamed from MX_.>; footprint (none) -> MX_Alps_Hybrid:MX-1U-NoLED
- MX_/1: renamed from MX_/?; footprint (none) -> MX_Alps_Hybrid:MX-1U-NoLED
- MX_0)1: renamed from MX_0); footprint (none) -> MX_Alps_Hybrid:MX-1U-NoLED
- MX_1!1: renamed from MX_1!; footprint (none) -> MX_Alps_Hybrid:MX-1U-NoLED
- MX_2@1: renamed from MX_2@; footprint (none) -> MX_Alps_Hybrid:MX-1U-NoLED
- MX_3#1: renamed from MX_3#; footprint (none) -> MX_Alps_Hybrid:MX-1U-NoLED
- MX_4$1: renamed from MX_4$; footprint (none) -> MX_Alps_Hybrid:MX-1U-NoLED
- MX_5%1: renamed from MX_5%; footprint (none) -> MX_Alps_Hybrid:MX-1U-NoLED
- MX_6^1: renamed from MX_6^; footprint (none) -> MX_Alps_Hybrid:MX-1U-NoLED
- MX_7&1: renamed from MX_7&; footprint (none) -> MX_Alps_Hybrid:MX-1U-NoLED
- MX_8*1: renamed from MX_8*; footprint (none) -> MX_Alps_Hybrid:MX-1U-NoLED
- MX_9(1: renamed from MX_9(; footprint (none) -> MX_Alps_Hybrid:MX-1U-NoLED
- MX_;:1: renamed from MX_;:; footprint (none) -> MX_Alps_Hybrid:MX-1U-NoLED
- MX_=+1: renamed from MX_=+; footprint (none) -> MX_Alps_Hybrid:MX-1U-NoLED
- MX_A1: renamed from MX_A; footprint (none) -> MX_Alps_Hybrid:MX-1U-NoLED
- MX_B1: renamed from MX_B; footprint (none) -> MX_Alps_Hybrid:MX-1U-NoLED
- MX_BKSPC1: renamed from MX_BKSPC; footprint (none) -> MX_Alps_Hybrid:MX-2U-NoLED
- MX_C1: renamed from MX_C; footprint (none) -> MX_Alps_Hybrid:MX-1U-NoLED
- MX_CAPS1: renamed from MX_CAPS; footprint (none) -> MX_Alps_Hybrid:MX-1.75U-NoLED
- MX_D1: renamed from MX_D; footprint (none) -> MX_Alps_Hybrid:MX-1U-NoLED
- MX_DEL1: renamed from MX_DEL; footprint (none) -> MX_Alps_Hybrid:MX-1.5U-NoLED
- MX_DOWN1: renamed from MX_DOWN; footprint (none) -> MX_Alps_Hybrid:MX-1U-NoLED
- MX_E1: renamed from MX_E; footprint (none) -> MX_Alps_Hybrid:MX-1U-NoLED
- MX_END1: renamed from MX_END; footprint (none) -> MX_Alps_Hybrid:MX-1U-NoLED
- MX_ENTER1: renamed from MX_ENTER; footprint (none) -> MX_Alps_Hybrid:MX-2.25U-NoLED
- MX_ESC1: renamed from MX_ESC; footprint (none) -> MX_Alps_Hybrid:MX-1.5U-NoLED
- MX_F1, MX_F10, MX_F11, MX_F12, MX_F2, MX_F3, MX_F4, MX_F5, MX_F6, MX_F7, MX_F8, MX_F9: footprint (none) -> MX_Alps_Hybrid:MX-1U-NoLED
- MX_F13: renamed from MX_F; footprint (none) -> MX_Alps_Hybrid:MX-1U-NoLED
- MX_FN1: renamed from MX_FN; footprint (none) -> MX_Alps_Hybrid:MX-1U-NoLED
- MX_G1: renamed from MX_G; footprint (none) -> MX_Alps_Hybrid:MX-1U-NoLED
- MX_GRV1: renamed from MX_GRV; footprint (none) -> MX_Alps_Hybrid:MX-1U-NoLED
- MX_H1: renamed from MX_H; footprint (none) -> MX_Alps_Hybrid:MX-1U-NoLED
- MX_HOME1: renamed from MX_HOME; footprint (none) -> MX_Alps_Hybrid:MX-1U-NoLED
- MX_I1: renamed from MX_I; footprint (none) -> MX_Alps_Hybrid:MX-1U-NoLED
- MX_J1: renamed from MX_J; footprint (none) -> MX_Alps_Hybrid:MX-1U-NoLED
- MX_K1: renamed from MX_K; footprint (none) -> MX_Alps_Hybrid:MX-1U-NoLED
- MX_L1: renamed from MX_L; footprint (none) -> MX_Alps_Hybrid:MX-1U-NoLED
- MX_LALT1, MX_LALT2: renamed from MX_LALT; footprint (none) -> MX_Alps_Hybrid:MX-1.25U-NoLED
- MX_LCTRL1: renamed from MX_LCTRL; footprint (none) -> MX_Alps_Hybrid:MX-1.25U-NoLED
- MX_LEFT1: renamed from MX_LEFT; footprint (none) -> MX_Alps_Hybrid:MX-1U-NoLED
- MX_LSHIFT1: renamed from MX_LSHIFT; footprint (none) -> MX_Alps_Hybrid:MX-2.25U-NoLED
- MX_LWIN1: renamed from MX_LWIN; footprint (none) -> MX_Alps_Hybrid:MX-1.25U-NoLED
- MX_M1: renamed from MX_M; footprint (none) -> MX_Alps_Hybrid:MX-1U-NoLED
- MX_N1: renamed from MX_N; footprint (none) -> MX_Alps_Hybrid:MX-1U-NoLED
- MX_O1: renamed from MX_O; footprint (none) -> MX_Alps_Hybrid:MX-1U-NoLED
- MX_P1: renamed from MX_P; footprint (none) -> MX_Alps_Hybrid:MX-1U-NoLED
- MX_PGDN1: renamed from MX_PGDN; footprint (none) -> MX_Alps_Hybrid:MX-1U-NoLED
- MX_PGUP1: renamed from MX_PGUP; footprint (none) -> MX_Alps_Hybrid:MX-1U-NoLED
- MX_Pn1: renamed from MX_Pn; footprint (none) -> MX_Alps_Hybrid:MX-1U-NoLED
- MX_Q1: renamed from MX_Q; footprint (none) -> MX_Alps_Hybrid:MX-1U-NoLED
- MX_R1: renamed from MX_R; footprint (none) -> MX_Alps_Hybrid:MX-1U-NoLED
- MX_RCTRL1: renamed from MX_RCTRL; footprint (none) -> MX_Alps_Hybrid:MX-1.25U-NoLED
- MX_RIGHT1: renamed from MX_RIGHT; footprint (none) -> MX_Alps_Hybrid:MX-1U-NoLED
- MX_RSHIFT1: renamed from MX_LSHIFT; footprint (none) -> MX_Alps_Hybrid:MX-1.75U-NoLED
- MX_S1: renamed from MX_S; footprint (none) -> MX_Alps_Hybrid:MX-1U-NoLED
- MX_SPC1: renamed from MX_SPC; footprint (none) -> MX_Alps_Hybrid:MX-6.25U-NoLED
- MX_T1: renamed from MX_T; footprint (none) -> MX_Alps_Hybrid:MX-1U-NoLED
- MX_TAB1: renamed from MX_TAB; footprint (none) -> MX_Alps_Hybrid:MX-1.5U-NoLED
- MX_U1: renamed from MX_U; footprint (none) -> MX_Alps_Hybrid:MX-1U-NoLED
- MX_UP1: renamed from MX_UP; footprint (none) -> MX_Alps_Hybrid:MX-1U-NoLED
- MX_V1: renamed from MX_V; footprint (none) -> MX_Alps_Hybrid:MX-1U-NoLED
- MX_W1: renamed from MX_W; footprint (none) -> MX_Alps_Hybrid:MX-1U-NoLED
- MX_X1: renamed from MX_X; footprint (none) -> MX_Alps_Hybrid:MX-1U-NoLED
- MX_Y1: renamed from MX_Y; footprint (none) -> MX_Alps_Hybrid:MX-1U-NoLED
- MX_Z1: renamed from MX_Z; footprint (none) -> MX_Alps_Hybrid:MX-1U-NoLED
- MX_[{1: renamed from MX_[{; footprint (none) -> MX_Alps_Hybrid:MX-1U-NoLED
- MX_\|1: renamed from MX_\|; footprint (none) -> MX_Alps_Hybrid:MX-1U-NoLED
- MX_]}1: renamed from MX_]}; footprint (none) -> MX_Alps_Hybrid:MX-1U-NoLED
- SW1: renamed from SW?; footprint (none) -> random-keyboard-parts:PushButton_6x6mm_TH_Pretty
- U1: renamed from U?; footprint (none) -> Keebio-Parts:Elite-C
- USB1: renamed from USB?; footprint (none) -> Keebio-Parts:USB-Mini-B_ LCSC-C46398
