File: cortex-face-1.kicad_pcb (KiCad board)
At the start: 2 copper layers, 94 parts

Commit message: Edge Cuts & DRC Errors Fixed
Other:
- rule trace_min: 0.2 -> 0.254
Changed lines of the file:
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@@
   (general
     (thickness 1.6)
-    (drawings 4)
-    (tracks 759)
+    (drawings 8)
+    (tracks 758)
     (zones 0)
     (modules 180)
@@
     (zone_clearance 0.508)
     (zone_45_only no)
-    (trace_min 0.2)
+    (trace_min 0.254)
     (via_size 0.8)
     (via_drill 0.4)
@@
       (net 2 ROW0))
   )
-  (gr_arc (start 54.51475 79.8195) (end 54.51475 76.0095) (angle -90) (layer Edge.Cuts) (width 0.12))
-  (gr_arc (start 54.51475 186.4995) (end 50.70475 186.4995) (angle -90) (layer Edge.Cuts) (width 0.12))
-  (gr_arc (start 351.69475 186.4995) (end 351.69475 190.3095) (angle -90) (layer Edge.Cuts) (width 0.12))
-  (gr_arc (start 351.69475 79.8195) (end 355.50475 79.8195) (angle -90) (layer Edge.Cuts) (width 0.12))
+  (gr_line (start 54.61 75.946) (end 351.536 75.946) (layer Edge.Cuts) (width 0.05))
+  (gr_line (start 50.673 186.309) (end 50.546 80.01) (layer Edge.Cuts) (width 0.05))
+  (gr_line (start 351.536 190.373) (end 54.737 190.373) (layer Edge.Cuts) (width 0.05))
+  (gr_line (start 355.6 80.01) (end 355.6 186.309) (layer Edge.Cuts) (width 0.05))
+  (gr_arc (start 351.536 80.01) (end 355.6 80.01) (angle -90) (layer Edge.Cuts) (width 0.05))
+  (gr_arc (start 351.536 186.309) (end 351.536 190.373) (angle -90) (layer Edge.Cuts) (width 0.05))
+  (gr_arc (start 54.737 186.309) (end 50.673 186.309) (angle -90) (layer Edge.Cuts) (width 0.05))
+  (gr_arc (start 54.61 80.01) (end 54.61 75.946) (angle -90) (layer Edge.Cuts) (width 0.05))
   (segment (start 96.74225 89.3445) (end 95.58945 89.3445) (width 0.254) (layer F.Cu) (net 1))
   (segment (start 95.58945 89.3445) (end 94.31945 90.6145) (width 0.254) (layer F.Cu) (net 1))
@@
   (segment (start 172.94275 81.7245) (end 176.11675 81.7245) (width 0.254) (layer F.Cu) (net 2))
   (segment (start 138.01675 81.7245) (end 172.94275 81.7245) (width 0.254) (layer F.Cu) (net 2))
-  (segment (start 59.81505 108.3542) (end 59.81505 119.7604) (width 0.254) (layer F.Cu) (net 2))
-  (segment (start 60.48375 107.7595) (end 59.81505 108.3542) (width 0.254) (layer F.Cu) (net 2))
-  (segment (start 62.550651 104.685397) (end 62.550651 105.692599) (width 0.254) (layer F.Cu) (net 2))
-  (segment (start 67.614049 99.621999) (end 62.550651 104.685397) (width 0.254) (layer F.Cu) (net 2))
-  (segment (start 62.550651 105.692599) (end 60.48375 107.7595) (width 0.254) (layer F.Cu) (net 2))
-  (segment (start 88.694852 99.6315) (end 75.08875 99.6315) (width 0.254) (layer F.Cu) (net 2))
-  (segment (start 98.32975 89.996602) (end 88.694852 99.6315) (width 0.254) (layer F.Cu) (net 2))
   (segment (start 99.91725 81.7245) (end 98.32975 81.7245) (width 0.254) (layer F.Cu) (net 2))
   (segment (start 98.32975 81.7245) (end 96.74225 81.7245) (width 0.254) (layer F.Cu) (net 2))
-  (segment (start 75.08875 99.6315) (end 67.614049 99.621999) (width 0.254) (layer F.Cu) (net 2))
+  (segment (start 56.92775 122.6185) (end 56.80075 122.7455) (width 0.254) (layer F.Cu) (net 2))
+  (segment (start 98.32975 83.312) (end 98.32975 89.996602) (width 0.254) (layer F.Cu) (net 2))
+  (segment (start 62.550651 104.685397) (end 62.550651 105.692599) (width 0.254) (layer F.Cu) (net 2))
   (segment (start 96.74225 81.7245) (end 98.32975 83.312) (width 0.254) (layer F.Cu) (net 2))
-  (segment (start 98.32975 83.312) (end 98.32975 84.0105) (width 0.254) (layer F.Cu) (net 2))
-  (segment (start 98.32975 84.0105) (end 98.32975 89.996602) (width 0.254) (layer F.Cu) (net 2))
-  (segment (start 56.80075 122.7455) (end 56.92775 122.6185) (width 0.254) (layer F.Cu) (net 2))
-  (segment (start 56.92775 122.6185) (end 59.81505 119.7604) (width 0.254) (layer F.Cu) (net 2))
-  (segment (start 56.80075 157.7975) (end 56.80075 122.7455) (width 0.254) (layer F.Cu) (net 2))
+  (segment (start 98.32975 89.996602) (end 88.9 99.441) (width 0.254) (layer F.Cu) (net 2))
+  (segment (start 88.9 99.441) (end 67.691 99.441) (width 0.254) (layer F.Cu) (net 2))
+  (segment (start 56.80075 122.7455) (end 56.80075 157.7975) (width 0.254) (layer F.Cu) (net 2))
+  (segment (start 60.48375 107.7595) (end 59.81505 108.3542) (width 0.254) (layer F.Cu) (net 2))
+  (segment (start 67.691 99.441) (end 67.31 99.822) (width 0.254) (layer F.Cu) (net 2))
+  (segment (start 67.31 99.822) (end 62.550651 104.685397) (width 0.254) (layer F.Cu) (net 2))
+  (segment (start 62.550651 105.692599) (end 60.48375 107.7595) (width 0.254) (layer F.Cu) (net 2))
+  (segment (start 59.81505 108.3542) (end 59.81505 119.7604) (width 0.254) (layer F.Cu) (net 2))
+  (segment (start 59.81505 119.7604) (end 56.92775 122.6185) (width 0.254) (layer F.Cu) (net 2))
   (segment (start 99.91725 89.3445) (end 104.04475 89.3445) (width 0.254) (layer F.Cu) (net 3))
   (segment (start 104.04475 89.3445) (end 105.31475 90.6145) (width 0.254) (layer F.Cu) (net 3))

Commit message: Updated footprints
Changed to USB micro for drop-in compatibility, changed connector wire size. No DRC errors.
Parts:
- added D1: D_Small, Keebio-Parts:Diode, F.Cu at (98.3, 85.5)
- added J1: Conn_01x04, Connector_Wire:SolderWirePad_1x04_P3.175mm_Drill0.8mm, B.Cu at (83.3, 95.1)
- added USB1: Molex-0548190589, Connector_USB:USB_Micro-B_GCT_USB3076-30-A, B.Cu at (78.5, 78.7)
- moved D10 1.59 mm to (334.9, 85.5)
- moved H10 1.59 mm to (338.0, 152.2)
- moved MX_-_1 1.59 mm to (271.4, 104.6)
- moved MX_=+1 1.59 mm to (290.4, 104.6)
- moved MX_BAR1 1.59 mm to (323.8, 123.6)
- moved MX_BKSPC1 1.59 mm to (319.0, 104.6)
- moved MX_FN1 1.59 mm to (271.4, 180.8)
- moved MX_Pn1 1.59 mm to (319.0, 85.5)
- moved MX_RCTRL1 1.59 mm to (290.4, 180.8)
- moved H5 1.59 mm to (204.7, 95.1)
- moved H7 1.59 mm to (240.4, 182.4)
- moved MX_,<1 1.59 mm to (238.0, 161.7)
- moved MX_0)1 1.59 mm to (252.3, 104.6)
- moved MX_3#1 1.59 mm to (119.0, 104.6)
- moved MX_5%1 1.59 mm to (157.1, 104.6)
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