File: _autosave-cortex-face-1.sch (KiCad schematic (older format))
At the start: 178 parts, among them J1 Conn_01x04, SW1 SW_Push, U1 Elite-C

Commit message: Sizing/Edge Cut Adjustments
Re-measured PCB and cut down PCB accordingly. Changed holes on edges to edge cuts
Parts:
- removed H6: Hole, MountingHole:MountingHole_6mm, symbol keebio:Hole
- renumbered H7 to H6, H8 to H7
Other:
- moved on the sheet: H6, H7
Changed lines of the file:
@@
 $EndComp
 $Comp
-L keebio:Hole H7
+L keebio:Hole H6
 U 1 1 5E01E2A7
-P 3000 1500
-F 0 "H7" H 3186 1553 60  0000 L CNN
-F 1 "Hole" H 3186 1447 60  0000 L CNN
-F 2 "MountingHole:MountingHole_6mm" H 3000 1500 60  0001 C CNN
-F 3 "" H 3000 1500 60  0001 C CNN
-	1    3000 1500
+P 2500 2000
+F 0 "H6" H 2686 2053 60  0000 L CNN
+F 1 "Hole" H 2686 1947 60  0000 L CNN
+F 2 "MountingHole:MountingHole_6mm" H 2500 2000 60  0001 C CNN
+F 3 "" H 2500 2000 60  0001 C CNN
+	1    2500 2000
 	1    0    0    -1
 $EndComp
@@
 $EndComp
 $Comp
-L keebio:Hole H6
-U 1 1 5E04EBB3
-P 2500 2000
-F 0 "H6" H 2686 2053 60  0000 L CNN
-F 1 "Hole" H 2686 1947 60  0000 L CNN
-F 2 "MountingHole:MountingHole_6mm" H 2500 2000 60  0001 C CNN
-F 3 "" H 2500 2000 60  0001 C CNN
-	1    2500 2000
+L keebio:Hole H7
+U 1 1 5E04EBB9
+P 3000 1500
+F 0 "H7" H 3186 1553 60  0000 L CNN
+F 1 "Hole" H 3186 1447 60  0000 L CNN
+F 2 "MountingHole:MountingHole_6mm" H 3000 1500 60  0001 C CNN
+F 3 "" H 3000 1500 60  0001 C CNN
+	1    3000 1500
 	1    0    0    -1
 $EndComp
-$Comp
-L keebio:Hole H8
-U 1 1 5E04EBB9
-P 3000 2000
-F 0 "H8" H 3186 2053 60  0000 L CNN
-F 1 "Hole" H 3186 1947 60  0000 L CNN
-F 2 "MountingHole:MountingHole_6mm" H 3000 2000 60  0001 C CNN
-F 3 "" H 3000 2000 60  0001 C CNN
-	1    3000 2000
-	1    0    0    -1
-$EndComp
