File: _autosave-bear-face-1.kicad_pcb (KiCad board)
At the start: 2 copper layers, 301.7 x 112.6 mm, 177 parts, among them J1 Conn_01x04, SW1 SW_Push

Commit message: Matrix, footprints changed
Changed to pure rectangular matrix, updated switch and diode SilkS, anticipate using on-board 32u4
Parts:
- removed J1: Conn_01x04, Connector_Wire:SolderWirePad_1x04_P3.175mm_Drill0.8mm
Connections:
- D1 pad 1: Net-(D1-Pad1) -> ROW0
- D10 pad 1: Net-(D10-Pad1) -> ROW0
- D11 pad 1: Net-(D11-Pad1) -> ROW0
- D12 pad 1: Net-(D12-Pad1) -> ROW0
- D13 pad 1: Net-(D13-Pad1) -> ROW0
- D14 pad 1: Net-(D14-Pad1) -> ROW0
- D15 pad 1: Net-(D15-Pad1) -> ROW0
- D16 pad 1: Net-(D16-Pad1) -> ROW1
- D17 pad 1: Net-(D17-Pad1) -> ROW1
- D18 pad 1: Net-(D18-Pad1) -> ROW1
- D19 pad 1: Net-(D19-Pad1) -> ROW1
- D2 pad 1: Net-(D2-Pad1) -> ROW0
- D20 pad 1: Net-(D20-Pad1) -> ROW1
- D21 pad 1: Net-(D21-Pad1) -> ROW1
- D22 pad 1: Net-(D22-Pad1) -> ROW1
- D23 pad 1: Net-(D23-Pad1) -> ROW1
- D24 pad 1: Net-(D24-Pad1) -> ROW1
- D25 pad 1: Net-(D25-Pad1) -> ROW1
- D26 pad 1: Net-(D26-Pad1) -> ROW1
- D27 pad 1: Net-(D27-Pad1) -> ROW1
- D28 pad 1: Net-(D28-Pad1) -> ROW1
- D29 pad 1: Net-(D29-Pad1) -> ROW1
- D3 pad 1: Net-(D3-Pad1) -> ROW0
- D30 pad 1: Net-(D30-Pad1) -> ROW1
- D31 pad 1: Net-(D31-Pad1) -> ROW2
- D32 pad 1: Net-(D32-Pad1) -> ROW2
- D33 pad 1: Net-(D33-Pad1) -> ROW2
- D34 pad 1: Net-(D34-Pad1) -> ROW2
- D35 pad 1: Net-(D35-Pad1) -> ROW2
- D36 pad 1: Net-(D36-Pad1) -> ROW2
- D37 pad 1: Net-(D37-Pad1) -> ROW2
- D38 pad 1: Net-(D38-Pad1) -> ROW2
- D39 pad 1: Net-(D39-Pad1) -> ROW2
- D4 pad 1: Net-(D4-Pad1) -> ROW0
- D40 pad 1: Net-(D40-Pad1) -> ROW2
- D41 pad 1: Net-(D41-Pad1) -> ROW2
- D42 pad 1: Net-(D42-Pad1) -> ROW2
- D43 pad 1: Net-(D43-Pad1) -> ROW2
- D44 pad 1: Net-(D44-Pad1) -> ROW2
- D45 pad 1: Net-(D45-Pad1) -> ROW2
- D46 pad 1: Net-(D46-Pad1) -> ROW3
- D47 pad 1: Net-(D47-Pad1) -> ROW3
- D48 pad 1: Net-(D48-Pad1) -> ROW3
- D49 pad 1: Net-(D49-Pad1) -> ROW3
- D5 pad 1: Net-(D5-Pad1) -> ROW0
- D50 pad 1: Net-(D50-Pad1) -> ROW3
- D51 pad 1: Net-(D51-Pad1) -> ROW3
- D52 pad 1: Net-(D52-Pad1) -> ROW3
- D53 pad 1: Net-(D53-Pad1) -> ROW3
- D54 pad 1: Net-(D54-Pad1) -> ROW3
- D55 pad 1: Net-(D55-Pad1) -> ROW3
- D56 pad 1: Net-(D56-Pad1) -> ROW3
- D57 pad 1: Net-(D57-Pad1) -> ROW3
- D58 pad 1: Net-(D58-Pad1) -> ROW3
- D59 pad 1: Net-(D59-Pad1) -> ROW3
- D6 pad 1: Net-(D6-Pad1) -> ROW0
- D60 pad 1: Net-(D60-Pad1) -> ROW4
- D61 pad 1: Net-(D61-Pad1) -> ROW4
- D62 pad 1: Net-(D62-Pad1) -> ROW4
- D63 pad 1: Net-(D63-Pad1) -> ROW4
- D64 pad 1: Net-(D64-Pad1) -> ROW4
- D65 pad 1: Net-(D65-Pad1) -> ROW4
- D66 pad 1: Net-(D66-Pad1) -> ROW4
- D67 pad 1: Net-(D67-Pad1) -> ROW4
- D68 pad 1: Net-(D68-Pad1) -> ROW4
- D69 pad 1: Net-(D69-Pad1) -> ROW4
- D7 pad 1: Net-(D7-Pad1) -> ROW0
- D70 pad 1: Net-(D70-Pad1) -> ROW4
- D71 pad 1: Net-(D71-Pad1) -> ROW4
- D72 pad 1: Net-(D72-Pad1) -> ROW4
- D73 pad 1: Net-(D73-Pad1) -> ROW4
- D74 pad 1: Net-(D74-Pad1) -> ROW5
- D75 pad 1: Net-(D75-Pad1) -> ROW5
- D76 pad 1: Net-(D76-Pad1) -> ROW5
- D77 pad 1: Net-(D77-Pad1) -> ROW5
- D78 pad 1: Net-(D78-Pad1) -> ROW5
- D79 pad 1: Net-(D79-Pad1) -> ROW5
- D8 pad 1: Net-(D8-Pad1) -> ROW0
- D80 pad 1: Net-(D80-Pad1) -> ROW5
- D81 pad 1: Net-(D81-Pad1) -> ROW5
- D82 pad 1: Net-(D82-Pad1) -> ROW5
- D83 pad 1: Net-(D83-Pad1) -> ROW5
- D9 pad 1: Net-(D9-Pad1) -> ROW0
- MX1 pad 1: Net-(MX1-Pad1) -> COL0
- MX10 pad 1: Net-(MX10-Pad1) -> COL9
- MX11 pad 1: Net-(MX11-Pad1) -> COL10
- MX12 pad 1: Net-(MX12-Pad1) -> COL11
- MX13 pad 1: Net-(MX13-Pad1) -> COL12
- MX14 pad 1: Net-(MX14-Pad1) -> COL13
- MX15 pad 1: Net-(MX15-Pad1) -> COL14
- MX16 pad 1: Net-(MX16-Pad1) -> COL0
- MX17 pad 1: Net-(MX17-Pad1) -> COL1
- MX18 pad 1: Net-(MX18-Pad1) -> COL2
- MX19 pad 1: Net-(MX19-Pad1) -> COL3
- MX2 pad 1: Net-(MX2-Pad1) -> COL1
- MX20 pad 1: Net-(MX20-Pad1) -> COL4
- MX21 pad 1: Net-(MX21-Pad1) -> COL5
- MX22 pad 1: Net-(MX22-Pad1) -> COL6
- MX23 pad 1: Net-(MX23-Pad1) -> COL7
- MX24 pad 1: Net-(MX24-Pad1) -> COL8
- MX25 pad 1: Net-(MX25-Pad1) -> COL9
- MX26 pad 1: Net-(MX26-Pad1) -> COL10
- MX27 pad 1: Net-(MX27-Pad1) -> COL11
- MX28 pad 1: Net-(MX28-Pad1) -> COL12
- MX29 pad 1: Net-(MX29-Pad1) -> COL13
- MX3 pad 1: Net-(MX3-Pad1) -> COL2
- MX30 pad 1: Net-(MX30-Pad1) -> COL14
- MX31 pad 1: Net-(MX31-Pad1) -> COL0
- MX32 pad 1: Net-(MX32-Pad1) -> COL1
- MX33 pad 1: Net-(MX33-Pad1) -> COL2
- MX34 pad 1: Net-(MX34-Pad1) -> COL3
- MX35 pad 1: Net-(MX35-Pad1) -> COL4
- MX36 pad 1: Net-(MX36-Pad1) -> COL5
- MX37 pad 1: Net-(MX37-Pad1) -> COL6
- MX38 pad 1: Net-(MX38-Pad1) -> COL7
- MX39 pad 1: Net-(MX39-Pad1) -> COL8
- MX4 pad 1: Net-(MX4-Pad1) -> COL3
- MX40 pad 1: Net-(MX40-Pad1) -> COL9
- MX41 pad 1: Net-(MX41-Pad1) -> COL10
- MX42 pad 1: Net-(MX42-Pad1) -> COL11
- MX43 pad 1: Net-(MX43-Pad1) -> COL12
- MX44 pad 1: Net-(MX44-Pad1) -> COL13
- MX45 pad 1: Net-(MX45-Pad1) -> COL14
- MX46 pad 1: Net-(MX46-Pad1) -> COL0
- MX47 pad 1: Net-(MX47-Pad1) -> COL1
- MX48 pad 1: Net-(MX48-Pad1) -> COL2
- MX49 pad 1: Net-(MX49-Pad1) -> COL3
- MX5 pad 1: Net-(MX5-Pad1) -> COL4
- MX50 pad 1: Net-(MX50-Pad1) -> COL4
- MX51 pad 1: Net-(MX51-Pad1) -> COL5
- MX52 pad 1: Net-(MX52-Pad1) -> COL6
- MX53 pad 1: Net-(MX53-Pad1) -> COL7
- MX54 pad 1: Net-(MX54-Pad1) -> COL8
- MX55 pad 1: Net-(MX55-Pad1) -> COL9
- MX56 pad 1: Net-(MX56-Pad1) -> COL10
- MX57 pad 1: Net-(MX57-Pad1) -> COL11
- MX58 pad 1: Net-(MX58-Pad1) -> COL13
- MX59 pad 1: Net-(MX59-Pad1) -> COL14
- MX6 pad 1: Net-(MX6-Pad1) -> COL5
- MX60 pad 1: Net-(MX60-Pad1) -> COL0
- MX61 pad 1: Net-(MX61-Pad1) -> COL1
- MX62 pad 1: Net-(MX62-Pad1) -> COL2
- MX63 pad 1: Net-(MX63-Pad1) -> COL3
- MX64 pad 1: Net-(MX64-Pad1) -> COL4
- MX65 pad 1: Net-(MX65-Pad1) -> COL5
- MX66 pad 1: Net-(MX66-Pad1) -> COL6
- MX67 pad 1: Net-(MX67-Pad1) -> COL7
- MX68 pad 1: Net-(MX68-Pad1) -> COL8
- MX69 pad 1: Net-(MX69-Pad1) -> COL9
- MX7 pad 1: Net-(MX7-Pad1) -> COL6
- MX70 pad 1: Net-(MX70-Pad1) -> COL10
- MX72 pad 1: Net-(MX72-Pad1) -> COL13
- MX73 pad 1: Net-(MX73-Pad1) -> COL14
- MX74 pad 1: Net-(MX74-Pad1) -> COL0
- MX75 pad 1: Net-(MX75-Pad1) -> COL1
- MX76 pad 1: Net-(MX76-Pad1) -> COL2
- MX77 pad 1: Net-(MX77-Pad1) -> COL5
- MX78 pad 1: Net-(MX78-Pad1) -> COL9
- MX79 pad 1: Net-(MX79-Pad1) -> COL10
- MX8 pad 1: Net-(MX8-Pad1) -> COL7
- MX81 pad 1: Net-(MX81-Pad1) -> Net-(MX71-Pad1)
- MX82 pad 1: Net-(MX82-Pad1) -> COL13
- MX83 pad 1: Net-(MX83-Pad1) -> COL14
- MX9 pad 1: Net-(MX9-Pad1) -> COL8
- USB1 pad 3: /D+ -> D+
- USB1 pad 4: /D- -> D-
- USB1 pad 5: /VCC -> VCC
Routing:
- net /VCC: track 15.6 -> 0.00 mm
- net GND: track 15.6 -> 0.00 mm
- net /D+: track 14.8 -> 0.00 mm
- net /D-: track 14.6 -> 0.00 mm
- net Net-(USB1-Pad6): track 13.9 -> 0.00 mm
