File: bear-face-1.kicad_pcb (KiCad board)
At the start: 2 copper layers, 301.7 x 112.6 mm, 178 parts, among them J1 Conn_01x04, SW1 SW_Push, U1 Elite-C

Commit message: Added ground fill
Ground filled entire board
Routing:
- added copper zone on B.Cu, net GND
Changed lines of the file:
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@@
   (segment (start 86.12575 70.621) (end 86.12575 72.785) (width 0.254) (layer B.Cu) (net 109) (status 20))
   (segment (start 84.93075 70.555) (end 86.05975 70.555) (width 0.254) (layer B.Cu) (net 109) (status 10))
+  (zone (net 93) (net_name GND) (layer B.Cu) (hatch edge 0.508)
+    (connect_pads (clearance 0.508))
+    (min_thickness 0.254)
+    (fill yes (arc_segments 32) (thermal_gap 0.508) (thermal_bridge_width 0.508))
+    (polygon
+      (pts
+        (xy 363.5375 183.35625) (xy 57.15 183.35625) (xy 57.15 67.46875) (xy 363.5375 67.46875)
+      )
+    )
+  )
 )

Commit message: SilkS added
Decoration
Parts:
- added G***: PASTA, bear_face_silks:pasta_small, B.Cu at (165.9, 116.7)
- added G***: FACE, bear_face_silks:cbf_small, B.Cu at (270.7, 128.6)

Commit message: Matrix, footprints changed
Changed to pure rectangular matrix, updated switch and diode SilkS, anticipate using on-board 32u4
Parts:
- removed G***: PASTA, bear_face_silks:pasta_small
- removed G***: FACE, bear_face_silks:cbf_small
- removed U1: Elite-C, Keebio-Parts:Elite-C
- moved MX1 0.06 mm to (72.2, 77.9)
- moved MX31 0.06 mm to (72.2, 116.0)
- moved MX15 0.06 mm to (348.4, 77.9)
- renumbered D11 to D1, D16 to D10, D17 to D11, D7 to D12, D8 to D13, D18 to D14, D10 to D15, D21 to D16, D22 to D17, D12 to D18, D23 to D19, D1 to D2, D14 to D20, D24 to D21, D33 to D22, D34 to D23, D25 to D24, D35 to D25, D36 to D28, D28 to D29, D2 to D3, D20 to D30, D30 to D31, D31 to D32, D40 to D33, D32 to D34, D41 to D35, D51 to D36, D42 to D37, D43 to D38, D52 to D39, D13 to D4, D44 to D40, D53 to D41, D45 to D42, D46 to D43, D37 to D44, D9 to D45, D39 to D46, D58 to D47, D49 to D48, D59 to D49, D3 to D5, D60 to D51, D70 to D52, D61 to D53, D71 to D54, D62 to D55, D63 to D56, D54 to D57, D55 to D58, D19 to D59, D4 to D6, D48 to D60, D67 to D61, D76 to D62, D68 to D63, D77 to D64, D69 to D65, D79 to D66, D80 to D67, D81 to D68, D72 to D69, D5 to D7, D73 to D70, D64 to D71, D29 to D72, D38 to D73, D57 to D74, D66 to D75, D75 to D76, D78 to D77, D82 to D78, D83 to D79, D15 to D8, D74 to D80, D65 to D81, D56 to D82, D47 to D83, D6 to D9, H3 to H2, H5 to H3, H7 to H4, H2 to H5, H4 to H6, H6 to H7, MX11 to MX1, MX16 to MX10, MX17 to MX11, MX7 to MX12, MX8 to MX13, MX18 to MX14, MX10 to MX15, MX21 to MX16, MX22 to MX17, MX12 to MX18, MX23 to MX19, MX1 to MX2, MX14 to MX20, MX24 to MX21, MX33 to MX22, MX34 to MX23, MX25 to MX24, MX35 to MX25, MX36 to MX28, MX28 to MX29, MX2 to MX3, MX20 to MX30, MX30 to MX31, MX31 to MX32, MX40 to MX33, MX32 to MX34, MX41 to MX35, MX51 to MX36, MX42 to MX37, MX43 to MX38, MX52 to MX39, MX13 to MX4, MX44 to MX40, MX53 to MX41, MX45 to MX42, MX46 to MX43, MX37 to MX44, MX9 to MX45, MX39 to MX46, MX58 to MX47, MX49 to MX48, MX59 to MX49, MX3 to MX5, MX60 to MX51, MX70 to MX52, MX61 to MX53, MX71 to MX54, MX62 to MX55, MX63 to MX56, MX54 to MX57, MX55 to MX58, MX19 to MX59, MX4 to MX6, MX48 to MX60, MX67 to MX61, MX76 to MX62, MX68 to MX63, MX77 to MX64, MX69 to MX65, MX79 to MX66, MX80 to MX67, MX81 to MX68, MX72 to MX69, MX5 to MX7, MX73 to MX70, MX64 to MX71, MX29 to MX72, MX38 to MX73, MX57 to MX74, MX66 to MX75, MX75 to MX76, MX78 to MX77, MX82 to MX78, MX83 to MX79, MX15 to MX8, MX74 to MX80, MX65 to MX81, MX56 to MX82, MX47 to MX83, MX6 to MX9
Connections:
- D1 pad 1: ROW1 -> Net-(D1-Pad1)
- D10 pad 1: ROW1 -> Net-(D10-Pad1)
- D11 pad 1: ROW1 -> Net-(D11-Pad1)
- D12 pad 1: ROW0 -> Net-(D12-Pad1)
- D13 pad 1: ROW0 -> Net-(D13-Pad1)
- D14 pad 1: ROW1 -> Net-(D14-Pad1)
- D15 pad 1: ROW0 -> Net-(D15-Pad1)
- D16 pad 1: ROW2 -> Net-(D16-Pad1)
- D17 pad 1: ROW2 -> Net-(D17-Pad1)
- D18 pad 1: ROW1 -> Net-(D18-Pad1)
- D19 pad 1: ROW2 -> Net-(D19-Pad1)
- D2 pad 1: ROW0 -> Net-(D2-Pad1)
- D20 pad 1: ROW1 -> Net-(D20-Pad1)
- D21 pad 1: ROW2 -> Net-(D21-Pad1)
- D22 pad 1: ROW3 -> Net-(D22-Pad1)
- D23 pad 1: ROW3 -> Net-(D23-Pad1)
- D24 pad 1: ROW2 -> Net-(D24-Pad1)
- D25 pad 1: ROW3 -> Net-(D25-Pad1)
- D26 pad 1: ROW2 -> Net-(D26-Pad1)
- D27 pad 1: ROW2 -> Net-(D27-Pad1)
- D28 pad 1: ROW3 -> Net-(D28-Pad1)
- D29 pad 1: ROW2 -> Net-(D29-Pad1)
- D3 pad 1: ROW0 -> Net-(D3-Pad1)
- D30 pad 1: ROW1 -> Net-(D30-Pad1)
- D31 pad 1: ROW3 -> Net-(D31-Pad1)
- D32 pad 1: ROW3 -> Net-(D32-Pad1)
- D33 pad 1: ROW4 -> Net-(D33-Pad1)
- D34 pad 1: ROW3 -> Net-(D34-Pad1)
- D35 pad 1: ROW4 -> Net-(D35-Pad1)
- D36 pad 1: ROW5 -> Net-(D36-Pad1)
- D37 pad 1: ROW4 -> Net-(D37-Pad1)
- D38 pad 1: ROW4 -> Net-(D38-Pad1)
- D39 pad 1: ROW5 -> Net-(D39-Pad1)
- D4 pad 1: ROW1 -> Net-(D4-Pad1)
- D40 pad 1: ROW4 -> Net-(D40-Pad1)
- D41 pad 1: ROW5 -> Net-(D41-Pad1)
- D42 pad 1: ROW4 -> Net-(D42-Pad1)
- D43 pad 1: ROW4 -> Net-(D43-Pad1)
- D44 pad 1: ROW3 -> Net-(D44-Pad1)
- D45 pad 1: ROW0 -> Net-(D45-Pad1)
- D46 pad 1: ROW4 -> Net-(D46-Pad1)
- D47 pad 1: ROW6 -> Net-(D47-Pad1)
- D48 pad 1: ROW5 -> Net-(D48-Pad1)
- D49 pad 1: ROW6 -> Net-(D49-Pad1)
- D5 pad 1: ROW0 -> Net-(D5-Pad1)
- D50 pad 1: ROW5 -> Net-(D50-Pad1)
- D51 pad 1: ROW6 -> Net-(D51-Pad1)
- D52 pad 1: ROW7 -> Net-(D52-Pad1)
- D53 pad 1: ROW6 -> Net-(D53-Pad1)
- D54 pad 1: ROW7 -> Net-(D54-Pad1)
- D55 pad 1: ROW6 -> Net-(D55-Pad1)
- D56 pad 1: ROW6 -> Net-(D56-Pad1)
- D57 pad 1: ROW5 -> Net-(D57-Pad1)
- D58 pad 1: ROW5 -> Net-(D58-Pad1)
- D59 pad 1: ROW1 -> Net-(D59-Pad1)
- D6 pad 1: ROW0 -> Net-(D6-Pad1)
- D60 pad 1: ROW5 -> Net-(D60-Pad1)
- D61 pad 1: ROW7 -> Net-(D61-Pad1)
- D62 pad 1: ROW8 -> Net-(D62-Pad1)
- D63 pad 1: ROW7 -> Net-(D63-Pad1)
- D64 pad 1: ROW8 -> Net-(D64-Pad1)
- D65 pad 1: ROW7 -> Net-(D65-Pad1)
- D66 pad 1: ROW8 -> Net-(D66-Pad1)
- D67 pad 1: ROW8 -> Net-(D67-Pad1)
- D68 pad 1: ROW8 -> Net-(D68-Pad1)
- D69 pad 1: ROW7 -> Net-(D69-Pad1)
- D7 pad 1: ROW0 -> Net-(D7-Pad1)
- D70 pad 1: ROW7 -> Net-(D70-Pad1)
- D71 pad 1: ROW6 -> Net-(D71-Pad1)
- D72 pad 1: ROW2 -> Net-(D72-Pad1)
- D73 pad 1: ROW3 -> Net-(D73-Pad1)
- D74 pad 1: ROW6 -> Net-(D74-Pad1)
- D75 pad 1: ROW7 -> Net-(D75-Pad1)
- D76 pad 1: ROW8 -> Net-(D76-Pad1)
- D77 pad 1: ROW8 -> Net-(D77-Pad1)
- D78 pad 1: ROW8 -> Net-(D78-Pad1)
- D79 pad 1: ROW8 -> Net-(D79-Pad1)
- D8 pad 1: ROW1 -> Net-(D8-Pad1)
- D80 pad 1: ROW7 -> Net-(D80-Pad1)
- D81 pad 1: ROW6 -> Net-(D81-Pad1)
- D82 pad 1: ROW5 -> Net-(D82-Pad1)
- D83 pad 1: ROW4 -> Net-(D83-Pad1)
- D9 pad 1: ROW0 -> Net-(D9-Pad1)
- MX1 pad 1: COL0 -> Net-(MX1-Pad1)
- MX10 pad 1: COL5 -> Net-(MX10-Pad1)
- MX11 pad 1: COL6 -> Net-(MX11-Pad1)
- MX12 pad 1: COL6 -> Net-(MX12-Pad1)
- MX13 pad 1: COL7 -> Net-(MX13-Pad1)
- MX14 pad 1: COL7 -> Net-(MX14-Pad1)
- MX15 pad 1: COL9 -> Net-(MX15-Pad1)
- MX16 pad 1: COL0 -> Net-(MX16-Pad1)
- MX17 pad 1: COL1 -> Net-(MX17-Pad1)
- MX18 pad 1: COL1 -> Net-(MX18-Pad1)
- MX19 pad 1: COL2 -> Net-(MX19-Pad1)
- MX2 pad 1: COL0 -> Net-(MX2-Pad1)
- MX20 pad 1: COL3 -> Net-(MX20-Pad1)
- MX21 pad 1: COL3 -> Net-(MX21-Pad1)
- MX22 pad 1: COL3 -> Net-(MX22-Pad1)
- MX23 pad 1: COL4 -> Net-(MX23-Pad1)
- MX24 pad 1: COL4 -> Net-(MX24-Pad1)
- MX25 pad 1: COL5 -> Net-(MX25-Pad1)
- MX26 pad 1: COL5 -> Net-(MX26-Pad1)
- MX27 pad 1: COL6 -> Net-(MX27-Pad1)
- MX28 pad 1: COL6 -> Net-(MX28-Pad1)
- MX29 pad 1: COL7 -> Net-(MX29-Pad1)
- MX3 pad 1: COL1 -> Net-(MX3-Pad1)
- MX30 pad 1: COL9 -> Net-(MX30-Pad1)
- MX31 pad 1: COL0 -> Net-(MX31-Pad1)
- MX32 pad 1: COL1 -> Net-(MX32-Pad1)
- MX33 pad 1: COL1 -> Net-(MX33-Pad1)
- MX34 pad 1: COL2 -> Net-(MX34-Pad1)
- MX35 pad 1: COL2 -> Net-(MX35-Pad1)
- MX36 pad 1: COL3 -> Net-(MX36-Pad1)
- MX37 pad 1: COL3 -> Net-(MX37-Pad1)
- MX38 pad 1: COL4 -> Net-(MX38-Pad1)
- MX39 pad 1: COL4 -> Net-(MX39-Pad1)
- MX4 pad 1: COL2 -> Net-(MX4-Pad1)
- MX40 pad 1: COL5 -> Net-(MX40-Pad1)
- MX41 pad 1: COL5 -> Net-(MX41-Pad1)
- MX42 pad 1: COL6 -> Net-(MX42-Pad1)
- MX43 pad 1: COL7 -> Net-(MX43-Pad1)
- MX44 pad 1: COL7 -> Net-(MX44-Pad1)
- MX45 pad 1: COL8 -> Net-(MX45-Pad1)
- MX46 pad 1: COL0 -> Net-(MX46-Pad1)
- MX47 pad 1: COL1 -> Net-(MX47-Pad1)
- MX48 pad 1: COL1 -> Net-(MX48-Pad1)
- MX49 pad 1: COL2 -> Net-(MX49-Pad1)
- MX5 pad 1: COL2 -> Net-(MX5-Pad1)
- MX50 pad 1: COL2 -> Net-(MX50-Pad1)
- MX51 pad 1: COL3 -> Net-(MX51-Pad1)
- MX52 pad 1: COL4 -> Net-(MX52-Pad1)
- MX53 pad 1: COL4 -> Net-(MX53-Pad1)
- MX54 pad 1: COL5 -> Net-(MX54-Pad1)
- MX55 pad 1: COL5 -> Net-(MX55-Pad1)
- MX56 pad 1: COL6 -> Net-(MX56-Pad1)
- MX57 pad 1: COL6 -> Net-(MX57-Pad1)
- MX58 pad 1: COL7 -> Net-(MX58-Pad1)
- MX59 pad 1: COL8 -> Net-(MX59-Pad1)
- MX6 pad 1: COL3 -> Net-(MX6-Pad1)
- MX60 pad 1: COL0 -> Net-(MX60-Pad1)
- MX61 pad 1: COL1 -> Net-(MX61-Pad1)
- MX62 pad 1: COL1 -> Net-(MX62-Pad1)
- MX63 pad 1: COL2 -> Net-(MX63-Pad1)
- MX64 pad 1: COL2 -> Net-(MX64-Pad1)
- MX65 pad 1: COL3 -> Net-(MX65-Pad1)
- MX66 pad 1: COL4 -> Net-(MX66-Pad1)
- MX67 pad 1: COL5 -> Net-(MX67-Pad1)
- MX68 pad 1: COL6 -> Net-(MX68-Pad1)
- MX69 pad 1: COL6 -> Net-(MX69-Pad1)
- MX7 pad 1: COL4 -> Net-(MX7-Pad1)
- MX70 pad 1: COL7 -> Net-(MX70-Pad1)
- MX71 pad 1: COL7 -> Net-(MX71-Pad1)
- MX72 pad 1: COL8 -> Net-(MX72-Pad1)
- MX73 pad 1: COL8 -> Net-(MX73-Pad1)
- MX74 pad 1: COL0 -> Net-(MX74-Pad1)
- MX75 pad 1: COL0 -> Net-(MX75-Pad1)
- MX76 pad 1: COL0 -> Net-(MX76-Pad1)
- MX77 pad 1: COL3 -> Net-(MX77-Pad1)
- MX78 pad 1: COL7 -> Net-(MX78-Pad1)
- MX79 pad 1: COL8 -> Net-(MX79-Pad1)
- MX8 pad 1: COL4 -> Net-(MX8-Pad1)
- MX80 pad 1: COL8 -> Net-(MX80-Pad1)
- MX81 pad 1: COL8 -> Net-(MX81-Pad1)
- MX82 pad 1: COL8 -> Net-(MX82-Pad1)
- MX83 pad 1: COL8 -> Net-(MX83-Pad1)
- MX9 pad 1: COL5 -> Net-(MX9-Pad1)
Routing:
- net ROW1: track 629.3 -> 0.00 mm
- net ROW2: track 524.0 -> 0.00 mm
- net ROW3: track 394.8 -> 0.00 mm
- net ROW0: track 387.5 -> 0.00 mm
- net ROW4: track 386.6 -> 0.00 mm
- net ROW5: track 366.8 -> 0.00 mm
- net ROW6: track 339.9 -> 0.00 mm
- net COL7: track 303.3 -> 0.00 mm
- net COL9: track 285.2 -> 0.00 mm
- net COL6: track 280.4 -> 0.00 mm
- net ROW7: track 278.9 -> 0.00 mm
- net COL8: track 270.0 -> 0.00 mm
- net COL5: track 259.5 -> 0.00 mm
- net COL4: track 241.9 -> 0.00 mm
- net ROW8: track 240.7 -> 0.00 mm
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
Commit message: MCU added, diodes changed
Changed to SMD components, matched components used in ai03's guide
Parts:
- removed J1: Conn_01x04, Connector_Wire:SolderWirePad_1x04_P3.175mm_Drill0.8mm
- added C1: 22pF, Capacitor_SMD:C_0805_2012Metric, F.Cu at (35.6, 82.0)
- added C2: 22pF, Capacitor_SMD:C_0805_2012Metric, F.Cu at (29.9, 89.8)
- added C3: 1uF, Capacitor_SMD:C_0805_2012Metric, F.Cu at (35.2, 85.3)
- added C4: 0.1uF, Capacitor_SMD:C_0805_2012Metric, F.Cu at (40.0, 82.0)
- added C5: 0.1uF, Capacitor_SMD:C_0805_2012Metric, F.Cu at (29.9, 92.7)
- added C6: 0.1uF, Capacitor_SMD:C_0805_2012Metric, F.Cu at (34.4, 89.8)
- added C7: 10uF, Capacitor_SMD:C_0805_2012Metric, F.Cu at (39.6, 85.0)
- added F1: 500mA, Fuse:Fuse_1206_3216Metric, F.Cu at (30.6, 82.2)
- added R1: 10k, Resistor_SMD:R_0805_2012Metric, F.Cu at (34.4, 92.7)
- added R2: 22, Resistor_SMD:R_0805_2012Metric, F.Cu at (38.8, 88.3)
- added R3: 22, Resistor_SMD:R_0805_2012Metric, F.Cu at (38.8, 91.2)
- added R4: 10k, Resistor_SMD:R_0805_2012Metric, F.Cu at (38.8, 94.2)
- added U1: ATmega32U4-AU, Package_QFP:TQFP-44_10x10mm_P0.8mm, F.Cu at (20.5, 87.8)
- added Y1: 16MHz, Crystal:Crystal_SMD_3225-4Pin_3.2x2.5mm, F.Cu at (30.4, 86.1)
- D1, D10, D11, D12, D13, D14, D15, D16, D17, D18, D19, D2, D20, D21, D22, D23, D24, D25, D26, D27, D28, D29, D3, D30, D31, D32, D33, D34, D35, D36, D37, D38, D39, D4, D40, D41, D42, D43, D44, D45, D46, D47, D48, D49, D5, D50, D51, D52, D53, D54, D55, D56, D57, D58, D59, D6, D60, D61, D62, D63, D64, D65, D66, D67, D68, D69, D7, D70, D71, D72, D73, D74, D75, D76, D77, D78, D79, D8, D80, D81, D82, D83, D9: footprint Keebio-Parts:Diode -> Diode_SMD:D_SOD-123
Connections:
- D1 pad 1: Net-(D1-Pad1) -> ROW0
- D10 pad 1: Net-(D10-Pad1) -> ROW0
- D11 pad 1: Net-(D11-Pad1) -> ROW0
- D12 pad 1: Net-(D12-Pad1) -> ROW0
- D13 pad 1: Net-(D13-Pad1) -> ROW0
- D14 pad 1: Net-(D14-Pad1) -> ROW0
- D15 pad 1: Net-(D15-Pad1) -> ROW0
- D16 pad 1: Net-(D16-Pad1) -> ROW1
- D17 pad 1: Net-(D17-Pad1) -> ROW1
- D18 pad 1: Net-(D18-Pad1) -> ROW1
- D19 pad 1: Net-(D19-Pad1) -> ROW1
- D2 pad 1: Net-(D2-Pad1) -> ROW0
- D20 pad 1: Net-(D20-Pad1) -> ROW1
- D21 pad 1: Net-(D21-Pad1) -> ROW1
- D22 pad 1: Net-(D22-Pad1) -> ROW1
- D23 pad 1: Net-(D23-Pad1) -> ROW1
- D24 pad 1: Net-(D24-Pad1) -> ROW1
- D25 pad 1: Net-(D25-Pad1) -> ROW1
- D26 pad 1: Net-(D26-Pad1) -> ROW1
- D27 pad 1: Net-(D27-Pad1) -> ROW1
- D28 pad 1: Net-(D28-Pad1) -> ROW1
- D29 pad 1: Net-(D29-Pad1) -> ROW1
- D3 pad 1: Net-(D3-Pad1) -> ROW0
- D30 pad 1: Net-(D30-Pad1) -> ROW1
- D31 pad 1: Net-(D31-Pad1) -> ROW2
- D32 pad 1: Net-(D32-Pad1) -> ROW2
- D33 pad 1: Net-(D33-Pad1) -> ROW2
- D34 pad 1: Net-(D34-Pad1) -> ROW2
- D35 pad 1: Net-(D35-Pad1) -> ROW2
- D36 pad 1: Net-(D36-Pad1) -> ROW2
- D37 pad 1: Net-(D37-Pad1) -> ROW2
- D38 pad 1: Net-(D38-Pad1) -> ROW2
- D39 pad 1: Net-(D39-Pad1) -> ROW2
- D4 pad 1: Net-(D4-Pad1) -> ROW0
- D40 pad 1: Net-(D40-Pad1) -> ROW2
- D41 pad 1: Net-(D41-Pad1) -> ROW2
- D42 pad 1: Net-(D42-Pad1) -> ROW2
- D43 pad 1: Net-(D43-Pad1) -> ROW2
- D44 pad 1: Net-(D44-Pad1) -> ROW2
- D45 pad 1: Net-(D45-Pad1) -> ROW2
- D46 pad 1: Net-(D46-Pad1) -> ROW3
- D47 pad 1: Net-(D47-Pad1) -> ROW3
- D48 pad 1: Net-(D48-Pad1) -> ROW3
- D49 pad 1: Net-(D49-Pad1) -> ROW3
- D5 pad 1: Net-(D5-Pad1) -> ROW0
- D50 pad 1: Net-(D50-Pad1) -> ROW3
- D51 pad 1: Net-(D51-Pad1) -> ROW3
- D52 pad 1: Net-(D52-Pad1) -> ROW3
- D53 pad 1: Net-(D53-Pad1) -> ROW3
- D54 pad 1: Net-(D54-Pad1) -> ROW3
- D55 pad 1: Net-(D55-Pad1) -> ROW3
- D56 pad 1: Net-(D56-Pad1) -> ROW3
- D57 pad 1: Net-(D57-Pad1) -> ROW3
- D58 pad 1: Net-(D58-Pad1) -> ROW3
- D59 pad 1: Net-(D59-Pad1) -> ROW3
- D6 pad 1: Net-(D6-Pad1) -> ROW0
- D60 pad 1: Net-(D60-Pad1) -> ROW4
- D61 pad 1: Net-(D61-Pad1) -> ROW4
- D62 pad 1: Net-(D62-Pad1) -> ROW4
- D63 pad 1: Net-(D63-Pad1) -> ROW4
- D64 pad 1: Net-(D64-Pad1) -> ROW4
- D65 pad 1: Net-(D65-Pad1) -> ROW4
- D66 pad 1: Net-(D66-Pad1) -> ROW4
- D67 pad 1: Net-(D67-Pad1) -> ROW4
- D68 pad 1: Net-(D68-Pad1) -> ROW4
- D69 pad 1: Net-(D69-Pad1) -> ROW4
- D7 pad 1: Net-(D7-Pad1) -> ROW0
- D70 pad 1: Net-(D70-Pad1) -> ROW4
- D71 pad 1: Net-(D71-Pad1) -> ROW4
- D72 pad 1: Net-(D72-Pad1) -> ROW4
- D73 pad 1: Net-(D73-Pad1) -> ROW4
- D74 pad 1: Net-(D74-Pad1) -> ROW5
- D75 pad 1: Net-(D75-Pad1) -> ROW5
- D76 pad 1: Net-(D76-Pad1) -> ROW5
- D77 pad 1: Net-(D77-Pad1) -> ROW5
- D78 pad 1: Net-(D78-Pad1) -> ROW5
- D79 pad 1: Net-(D79-Pad1) -> ROW5
- D8 pad 1: Net-(D8-Pad1) -> ROW0
- D80 pad 1: Net-(D80-Pad1) -> ROW5
- D81 pad 1: Net-(D81-Pad1) -> ROW5
- D82 pad 1: Net-(D82-Pad1) -> ROW5
- D83 pad 1: Net-(D83-Pad1) -> ROW5
- D9 pad 1: Net-(D9-Pad1) -> ROW0
- MX1 pad 1: Net-(MX1-Pad1) -> COL0
- MX10 pad 1: Net-(MX10-Pad1) -> COL9
- MX11 pad 1: Net-(MX11-Pad1) -> COL10
- MX12 pad 1: Net-(MX12-Pad1) -> COL11
- MX13 pad 1: Net-(MX13-Pad1) -> COL12
- MX14 pad 1: Net-(MX14-Pad1) -> COL13
- MX15 pad 1: Net-(MX15-Pad1) -> COL14
- MX16 pad 1: Net-(MX16-Pad1) -> COL0
- MX17 pad 1: Net-(MX17-Pad1) -> COL1
- MX18 pad 1: Net-(MX18-Pad1) -> COL2
- MX19 pad 1: Net-(MX19-Pad1) -> COL3
- MX2 pad 1: Net-(MX2-Pad1) -> COL1
- MX20 pad 1: Net-(MX20-Pad1) -> COL4
- MX21 pad 1: Net-(MX21-Pad1) -> COL5
- MX22 pad 1: Net-(MX22-Pad1) -> COL6
- MX23 pad 1: Net-(MX23-Pad1) -> COL7
- MX24 pad 1: Net-(MX24-Pad1) -> COL8
- MX25 pad 1: Net-(MX25-Pad1) -> COL9
- MX26 pad 1: Net-(MX26-Pad1) -> COL10
- MX27 pad 1: Net-(MX27-Pad1) -> COL11
- MX28 pad 1: Net-(MX28-Pad1) -> COL12
- MX29 pad 1: Net-(MX29-Pad1) -> COL13
- MX3 pad 1: Net-(MX3-Pad1) -> COL2
- MX30 pad 1: Net-(MX30-Pad1) -> COL14
- MX31 pad 1: Net-(MX31-Pad1) -> COL0
- MX32 pad 1: Net-(MX32-Pad1) -> COL1
- MX33 pad 1: Net-(MX33-Pad1) -> COL2
- MX34 pad 1: Net-(MX34-Pad1) -> COL3
- MX35 pad 1: Net-(MX35-Pad1) -> COL4
- MX36 pad 1: Net-(MX36-Pad1) -> COL5
- MX37 pad 1: Net-(MX37-Pad1) -> COL6
- MX38 pad 1: Net-(MX38-Pad1) -> COL7
- MX39 pad 1: Net-(MX39-Pad1) -> COL8
- MX4 pad 1: Net-(MX4-Pad1) -> COL3
- MX40 pad 1: Net-(MX40-Pad1) -> COL9
- MX41 pad 1: Net-(MX41-Pad1) -> COL10
- MX42 pad 1: Net-(MX42-Pad1) -> COL11
- MX43 pad 1: Net-(MX43-Pad1) -> COL12
- MX44 pad 1: Net-(MX44-Pad1) -> COL13
- MX45 pad 1: Net-(MX45-Pad1) -> COL14
- MX46 pad 1: Net-(MX46-Pad1) -> COL0
- MX47 pad 1: Net-(MX47-Pad1) -> COL1
- MX48 pad 1: Net-(MX48-Pad1) -> COL2
- MX49 pad 1: Net-(MX49-Pad1) -> COL3
- MX5 pad 1: Net-(MX5-Pad1) -> COL4
- MX50 pad 1: Net-(MX50-Pad1) -> COL4
- MX51 pad 1: Net-(MX51-Pad1) -> COL5
- MX52 pad 1: Net-(MX52-Pad1) -> COL6
- MX53 pad 1: Net-(MX53-Pad1) -> COL7
- MX54 pad 1: Net-(MX54-Pad1) -> COL8
- MX55 pad 1: Net-(MX55-Pad1) -> COL9
- MX56 pad 1: Net-(MX56-Pad1) -> COL10
- MX57 pad 1: Net-(MX57-Pad1) -> COL11
- MX58 pad 1: Net-(MX58-Pad1) -> COL13
- MX59 pad 1: Net-(MX59-Pad1) -> COL14
- MX6 pad 1: Net-(MX6-Pad1) -> COL5
- MX60 pad 1: Net-(MX60-Pad1) -> COL0
- MX61 pad 1: Net-(MX61-Pad1) -> COL1
- MX62 pad 1: Net-(MX62-Pad1) -> COL2
- MX63 pad 1: Net-(MX63-Pad1) -> COL3
- MX64 pad 1: Net-(MX64-Pad1) -> COL4
- MX65 pad 1: Net-(MX65-Pad1) -> COL5
- MX66 pad 1: Net-(MX66-Pad1) -> COL6
- MX67 pad 1: Net-(MX67-Pad1) -> COL7
- MX68 pad 1: Net-(MX68-Pad1) -> COL8
- MX69 pad 1: Net-(MX69-Pad1) -> COL9
- MX7 pad 1: Net-(MX7-Pad1) -> COL6
- MX70 pad 1: Net-(MX70-Pad1) -> COL10
- MX71 pad 1: Net-(MX71-Pad1) -> COL12
- MX72 pad 1: Net-(MX72-Pad1) -> COL13
- MX73 pad 1: Net-(MX73-Pad1) -> COL14
- MX74 pad 1: Net-(MX74-Pad1) -> COL0
- MX75 pad 1: Net-(MX75-Pad1) -> COL1
- MX76 pad 1: Net-(MX76-Pad1) -> COL2
- MX77 pad 1: Net-(MX77-Pad1) -> COL5
- MX78 pad 1: Net-(MX78-Pad1) -> COL9
- MX79 pad 1: Net-(MX79-Pad1) -> COL10
- MX8 pad 1: Net-(MX8-Pad1) -> COL7
- MX80 pad 1: Net-(MX80-Pad1) -> COL11
- MX81 pad 1: Net-(MX81-Pad1) -> COL12
- MX82 pad 1: Net-(MX82-Pad1) -> COL13
- MX83 pad 1: Net-(MX83-Pad1) -> COL14
- MX9 pad 1: Net-(MX9-Pad1) -> COL8
- SW1 pad 1: RESET -> GND
- SW1 pad 2: GND -> Net-(R1-Pad2)
- USB1 pad 3: /D+ -> D+
- USB1 pad 4: /D- -> D-
- USB1 pad 5: /VCC -> VCC
Routing:
- net /VCC: track 15.6 -> 0.00 mm
- net GND: track 15.6 -> 0.00 mm
- net /D+: track 14.8 -> 0.00 mm
- net /D-: track 14.6 -> 0.00 mm
- net Net-(USB1-Pad6): track 13.9 -> 0.00 mm

Commit message: South facing switches
Rotated switches to be south-facing and rotated diodes to match
Parts:
- D1, D10, D11, D12, D13, D14, D15, D16, D17, D18, D19, D2, D20, D21, D22, D23, D24, D25, D26, D27, D28, D29, D3, D30, D31, D32, D33, D34, D35, D36, D37, D38, D39, D4, D40, D41, D42, D43, D44, D45, D46, D47, D48, D49, D5, D50, D51, D52, D53, D54, D55, D56, D57, D58, D59, D6, D60, D61, D62, D63, D64, D65, D66, D67, D68, D69, D7, D70, D71, D72, D73, D74, D75, D76, D77, D78, D79, D8, D80, D81, D82, D83, D9: moved to B.Cu
- moved D71 23.3 mm to (292.5, 154.1), turned to 90 degrees
- moved D74 22.5 mm to (61.6, 173.0), turned to 90 degrees
- moved D76 18.6 mm to (106.8, 173.1)
- moved D36 16.2 mm to (180.5, 116.0), turned to 90 degrees
- moved D55 16.2 mm to (244.9, 135.0), turned to 90 degrees
- moved D11 16.2 mm to (259.2, 77.9), turned to 90 degrees
- moved D12 16.2 mm to (294.8, 77.9), turned to 90 degrees
- moved D13 16.2 mm to (297.3, 77.9), turned to 90 degrees
- moved D14 16.2 mm to (332.9, 77.9), turned to 90 degrees
- moved D35 16.2 mm to (144.9, 116.0), turned to 90 degrees
- moved D37 16.2 mm to (183.0, 116.0), turned to 90 degrees
- moved D38 16.2 mm to (218.6, 116.0), turned to 90 degrees
- moved D39 16.2 mm to (221.1, 116.0), turned to 90 degrees
- moved D41 16.2 mm to (259.2, 116.0), turned to 90 degrees
- moved D42 16.2 mm to (294.8, 116.0), turned to 90 degrees
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Other:
- board text removed: "Bear Face v1 by chemicalwill 01/06/2020"

Commit message: Diode footprints updated, MCU components started
Parts:
- C1, C2, C4, C5, C6, C7, U1, Y1: moved to B.Cu
- D1, D10, D11, D12, D13, D14, D15, D16, D17, D18, D19, D2, D20, D21, D22, D23, D24, D25, D26, D27, D28, D29, D3, D30, D31, D32, D33, D34, D35, D36, D37, D38, D39, D4, D40, D41, D42, D43, D44, D45, D46, D47, D48, D49, D5, D50, D51, D52, D53, D54, D55, D56, D57, D58, D59, D6, D60, D61, D62, D63, D64, D65, D66, D67, D68, D69, D7, D70, D71, D72, D73, D74, D75, D76, D77, D78, D79, D8, D80, D81, D82, D83, D9: footprint Diode_SMD:D_SOD-123 -> Bear-Face-1_parts:D_SOD-123
- MX77: footprint MX_Only:MXOnly-6.25U-NoLED -> MX_Only:MXOnly-6.25U-ReversedStabilizers-NoLED
- moved U1 160.4 mm to (158.0, 170.4)
- moved C5 157.2 mm to (168.2, 167.5), turned to 90 degrees
- moved C6 156.1 mm to (162.1, 179.4), turned to 180 degrees
- moved C7 148.2 mm to (153.8, 179.5)
- moved C1 148.2 mm to (161.9, 159.4), turned to 90 degrees
- moved Y1 147.2 mm to (157.9, 159.5), turned to 180 degrees
- moved C2 142.2 mm to (154.0, 159.4), turned to 270 degrees
- moved C4 139.4 mm to (147.6, 170.6), turned to 270 degrees
- moved C3 34.4 mm to (22.4, 117.2)
- moved R2 15.7 mm to (29.3, 100.9)
- moved R1 12.1 mm to (25.4, 100.9)
- moved R3 11.1 mm to (33.3, 100.9)
- moved R4 6.85 mm to (37.3, 100.9)
- turned D75 to 90 degrees
- turned D76 to 90 degrees

Commit message: Short diode tracks added
Parts:
- C3, F1, R1, R2, R3, R4: moved to B.Cu
- SW1: footprint random-keyboard-parts:PushButton_6x6mm_TH_Pretty -> random-keyboard-parts:SKQG-1155865
- moved R1 149.6 mm to (163.8, 157.5), turned to 180 degrees
- moved C3 140.0 mm to (156.2, 158.2), turned to 180 degrees
- moved R2 69.4 mm to (83.1, 56.9), turned to 90 degrees
- moved R4 61.9 mm to (80.8, 56.9), turned to 90 degrees
- moved R3 60.9 mm to (75.4, 56.9)
- moved F1 60.7 mm to (86.1, 57.7), turned to 90 degrees
- moved C2 19.6 mm to (167.6, 173.5), turned to 0 degrees
- moved C7 17.6 mm to (146.3, 163.6), turned to 270 degrees
- moved C6 16.4 mm to (146.3, 175.0), turned to 90 degrees
- moved C4 14.3 mm to (159.3, 178.8), turned to 0 degrees
- moved Y1 13.6 mm to (167.6, 168.9), turned to 90 degrees
- moved C5 7.65 mm to (163.8, 161.3), turned to 180 degrees
- moved C1 7.56 mm to (167.6, 164.3), turned to 180 degrees
- moved U1 2.49 mm to (155.9, 169.1), turned to 270 degrees
- moved SW1 1.12 mm to (84.9, 130.2)
Routing:
- net Net-(D71-Pad2): track 0.00 -> 19.8 mm
- net Net-(D60-Pad2): track 0.00 -> 19.5 mm
- net Net-(D58-Pad2): track 0.00 -> 19.5 mm
- net ROW2: track 0.00 -> 17.8 mm
- net ROW4: track 0.00 -> 17.8 mm
- net ROW1: track 0.00 -> 17.8 mm
- net ROW0: track 0.00 -> 17.8 mm
- net Net-(D15-Pad2): track 0.00 -> 17.4 mm
- net Net-(D29-Pad2): track 0.00 -> 17.1 mm
- net Net-(D76-Pad2): track 0.00 -> 15.9 mm
- net ROW3: track 0.00 -> 15.2 mm
- net Net-(D3-Pad2): track 0.00 -> 13.8 mm
- net Net-(D73-Pad2): track 0.00 -> 13.6 mm
- net Net-(D51-Pad2): track 0.00 -> 12.7 mm
- net Net-(D46-Pad2): track 0.00 -> 12.7 mm
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
Commit message: THT diodes and short tracks
Changed to use a combination of THT and SMD components
Parts:
- D1, D10, D11, D12, D13, D14, D15, D16, D17, D18, D19, D2, D20, D21, D22, D23, D24, D25, D26, D27, D28, D29, D3, D30, D31, D32, D33, D34, D35, D36, D37, D38, D39, D4, D40, D41, D42, D43, D44, D45, D46, D47, D48, D49, D5, D50, D51, D52, D53, D54, D55, D56, D57, D58, D59, D6, D60, D61, D62, D63, D64, D65, D66, D67, D68, D69, D7, D70, D71, D72, D73, D74, D75, D76, D77, D78, D79, D8, D80, D81, D82, D83, D9: footprint Bear-Face-1_parts:D_SOD-123 -> Keebio-Parts:Diode
- SW1: footprint random-keyboard-parts:SKQG-1155865 -> random-keyboard-parts:PushButton_6x6mm_TH_Pretty
- U1: footprint Package_QFP:TQFP-44_10x10mm_P0.8mm -> Keebio-Parts:ATMEGA32U4-AU
- moved R4 140.7 mm to (151.0, 178.8), turned to 0 degrees
- moved R3 28.4 mm to (85.2, 83.6), turned to 90 degrees
- moved R2 26.7 mm to (82.9, 83.6)
- moved F1 25.9 mm to (87.5, 83.6)
Routing:
- net ROW4: track 17.8 -> 5.08 mm
- net ROW5: track 10.2 -> 0.00 mm
- net Net-(D73-Pad2): track 13.6 -> 12.0 mm
- net Net-(D76-Pad2): track 15.9 -> 14.3 mm
- net Net-(D2-Pad2): track 9.14 -> 7.87 mm
- net Net-(D3-Pad2): track 13.8 -> 13.0 mm
- net Net-(D24-Pad2): track 7.55 -> 6.87 mm
- net Net-(D21-Pad2): track 12.6 -> 12.0 mm
- net Net-(D18-Pad2): track 7.55 -> 6.87 mm
- net Net-(D16-Pad2): track 7.55 -> 6.87 mm
- net Net-(D17-Pad2): track 12.6 -> 12.0 mm
- net Net-(D15-Pad2): track 17.4 -> 16.7 mm
- net Net-(D14-Pad2): track 7.55 -> 6.87 mm
- net Net-(D30-Pad2): track 12.6 -> 12.0 mm
- net Net-(D29-Pad2): track 17.1 -> 16.4 mm
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