File: bear-face-1.sch (KiCad schematic (older format))
At the start: 190 parts, among them J1 USB_B_Micro, SW1 SW_Push, U1 ATmega32U4-AU, Y1 16MHz

Commit message: Tracks finished, DRC check passed
Connections:
- net COL0: now also U1.39 (PF4)
- net COL1: now also U1.37 (PF6)
- net COL10: now also U1.22 (PD5)
- net COL11: now also U1.25 (PD4)
- net COL12: now also U1.26 (PD6)
- net COL13: now also U1.27 (PD7)
- net COL14: now also U1.28 (PB4)
- net COL2: now also U1.38 (PF5)
- net COL3: now also U1.41 (PF0)
- net COL4: now also U1.10 (PB2)
- net COL5: now also U1.12 (PB7)
- net COL6: now also U1.18 (PD0)
- net COL7: now also U1.19 (PD1)
- net COL8: now also U1.20 (PD2)
- net COL9: now also U1.21 (PD3)
- net ROW0: now also U1.9 (PB1)
- net ROW1: now also U1.1 (PE6)
- net ROW2: now also U1.8 (PB0)
- net ROW3: now also U1.11 (PB3)
- net ROW4: now also U1.40 (PF1)
- net ROW5: now also U1.36 (PF7)
- no-connect marks 0 -> 5
