File: bear_face_pcb.sch (KiCad schematic (older format))
At the start: 201 parts, among them J1 USB_B_Micro, J2 Conn_02x03_Odd_Even, Q1 2N7002, SW1 SW_Push, U1 ATmega32U4-AU, U2 SRV05-4, Y1 16MHz

Commit message: Changed LCSC# for crystal
Now basic part
Parts:
- Y1: LCSC# C89379 -> C13738
Changed lines of the file:
@@
 F 2 "Crystal:Crystal_SMD_3225-4Pin_3.2x2.5mm_HandSoldering" H 1250 4100 50  0001 C CNN
 F 3 "~" H 1250 4100 50  0001 C CNN
-F 4 "C89379" V 1250 4100 50  0001 C CNN "LCSC#"
+F 4 "C13738" V 1250 4100 50  0001 C CNN "LCSC#"
 	1    1250 4100
 	0    1    1    0

Commit message: Changed crystal footprint for SMT assembly
* Hand-solder footprint was too large
Parts:
- Y1: footprint Crystal:Crystal_SMD_3225-4Pin_3.2x2.5mm_HandSoldering -> Crystal:Crystal_SMD_3225-4Pin_3.2x2.5mm
Changed lines of the file:
@@
 F 0 "Y1" V 1204 4244 50  0000 L CNN
 F 1 "16MHz" V 1295 4244 50  0000 L CNN
-F 2 "Crystal:Crystal_SMD_3225-4Pin_3.2x2.5mm_HandSoldering" H 1250 4100 50  0001 C CNN
+F 2 "Crystal:Crystal_SMD_3225-4Pin_3.2x2.5mm" H 1250 4100 50  0001 C CNN
 F 3 "~" H 1250 4100 50  0001 C CNN
 F 4 "C13738" V 1250 4100 50  0001 C CNN "LCSC#"

Commit message: Changed hand-solder pads to... not hand-solder
Parts:
- C1, C2, C3, C4, C5, C6, C7: footprint Capacitor_SMD:C_0805_2012Metric_Pad1.15x1.40mm_HandSolder -> Capacitor_SMD:C_0805_2012Metric
- R1, R2, R3, R4, R5, R6: footprint Resistor_SMD:R_0805_2012Metric_Pad1.15x1.40mm_HandSolder -> Resistor_SMD:R_0805_2012Metric
Changed lines of the file:
@@
 F 0 "R1" V 1654 2400 50  0000 C CNN
 F 1 "22" V 1745 2400 50  0000 C CNN
-F 2 "Resistor_SMD:R_0805_2012Metric_Pad1.15x1.40mm_HandSolder" H 1850 2400 50  0001 C CNN
+F 2 "Resistor_SMD:R_0805_2012Metric" H 1850 2400 50  0001 C CNN
 F 3 "~" H 1850 2400 50  0001 C CNN
 F 4 "C17561" V 1850 2400 50  0001 C CNN "LCSC#"
@@
 F 0 "R2" V 1904 2500 50  0000 C CNN
 F 1 "22" V 1995 2500 50  0000 C CNN
-F 2 "Resistor_SMD:R_0805_2012Metric_Pad1.15x1.40mm_HandSolder" H 2100 2500 50  0001 C CNN
+F 2 "Resistor_SMD:R_0805_2012Metric" H 2100 2500 50  0001 C CNN
 F 3 "~" H 2100 2500 50  0001 C CNN
 F 4 "C17561" V 2100 2500 50  0001 C CNN "LCSC#"
@@
 F 0 "C3" H 1542 5246 50  0000 L CNN
 F 1 "1uF" H 1542 5155 50  0000 L CNN
-F 2 "Capacitor_SMD:C_0805_2012Metric_Pad1.15x1.40mm_HandSolder" H 1450 5200 50  0001 C CNN
+F 2 "Capacitor_SMD:C_0805_2012Metric" H 1450 5200 50  0001 C CNN
 F 3 "~" H 1450 5200 50  0001 C CNN
 F 4 "C28323" H 1450 5200 50  0001 C CNN "LCSC#"
@@
 F 0 "C4" H 3692 7246 50  0000 L CNN
 F 1 "100nF" H 3692 7155 50  0000 L CNN
-F 2 "Capacitor_SMD:C_0805_2012Metric_Pad1.15x1.40mm_HandSolder" H 3600 7200 50  0001 C CNN
+F 2 "Capacitor_SMD:C_0805_2012Metric" H 3600 7200 50  0001 C CNN
 F 3 "~" H 3600 7200 50  0001 C CNN
 F 4 "C49678" H 3600 7200 50  0001 C CNN "LCSC#"
@@
 F 0 "C5" H 4092 7246 50  0000 L CNN
 F 1 "100nF" H 4092 7155 50  0000 L CNN
-F 2 "Capacitor_SMD:C_0805_2012Metric_Pad1.15x1.40mm_HandSolder" H 4000 7200 50  0001 C CNN
+F 2 "Capacitor_SMD:C_0805_2012Metric" H 4000 7200 50  0001 C CNN
 F 3 "~" H 4000 7200 50  0001 C CNN
 F 4 "C49678" H 4000 7200 50  0001 C CNN "LCSC#"
@@
 F 0 "C6" H 4492 7246 50  0000 L CNN
 F 1 "100nF" H 4492 7155 50  0000 L CNN
-F 2 "Capacitor_SMD:C_0805_2012Metric_Pad1.15x1.40mm_HandSolder" H 4400 7200 50  0001 C CNN
+F 2 "Capacitor_SMD:C_0805_2012Metric" H 4400 7200 50  0001 C CNN
 F 3 "~" H 4400 7200 50  0001 C CNN
 F 4 "C49678" H 4400 7200 50  0001 C CNN "LCSC#"
@@
 F 0 "C7" H 4892 7246 50  0000 L CNN
 F 1 "10uF" H 4892 7155 50  0000 L CNN
-F 2 "Capacitor_SMD:C_0805_2012Metric_Pad1.15x1.40mm_HandSolder" H 4800 7200 50  0001 C CNN
+F 2 "Capacitor_SMD:C_0805_2012Metric" H 4800 7200 50  0001 C CNN
 F 3 "~" H 4800 7200 50  0001 C CNN
 F 4 "C15850" H 4800 7200 50  0001 C CNN "LCSC#"
@@
 F 0 "C1" V 621 3900 50  0000 C CNN
 F 1 "22pF" V 712 3900 50  0000 C CNN
-F 2 "Capacitor_SMD:C_0805_2012Metric_Pad1.15x1.40mm_HandSolder" H 850 3900 50  0001 C CNN
+F 2 "Capacitor_SMD:C_0805_2012Metric" H 850 3900 50  0001 C CNN
 F 3 "~" H 850 3900 50  0001 C CNN
 F 4 "C1804" V 850 3900 50  0001 C CNN "LCSC#"
@@
 F 0 "C2" V 621 4300 50  0000 C CNN
 F 1 "22pF" V 712 4300 50  0000 C CNN
-F 2 "Capacitor_SMD:C_0805_2012Metric_Pad1.15x1.40mm_HandSolder" H 850 4300 50  0001 C CNN
+F 2 "Capacitor_SMD:C_0805_2012Metric" H 850 4300 50  0001 C CNN
 F 3 "~" H 850 4300 50  0001 C CNN
 F 4 "C1804" V 850 4300 50  0001 C CNN "LCSC#"
@@
 F 0 "R6" H 8559 5796 50  0000 L CNN
 F 1 "10k" H 8559 5705 50  0000 L CNN
-F 2 "Resistor_SMD:R_0805_2012Metric_Pad1.15x1.40mm_HandSolder" H 8500 5750 50  0001 C CNN
+F 2 "Resistor_SMD:R_0805_2012Metric" H 8500 5750 50  0001 C CNN
 F 3 "~" H 8500 5750 50  0001 C CNN
 F 4 "C17414" H 8500 5750 50  0001 C CNN "LCSC#"
@@
 F 0 "R3" V 3254 5900 50  0000 C CNN
 F 1 "10k" V 3345 5900 50  0000 C CNN
-F 2 "Resistor_SMD:R_0805_2012Metric_Pad1.15x1.40mm_HandSolder" H 3450 5900 50  0001 C CNN
+F 2 "Resistor_SMD:R_0805_2012Metric" H 3450 5900 50  0001 C CNN
 F 3 "~" H 3450 5900 50  0001 C CNN
 F 4 "C17414" V 3450 5900 50  0001 C CNN "LCSC#"
@@
 F 0 "R4" H 5909 7146 50  0000 L CNN
 F 1 "4.7k" H 5909 7055 50  0000 L CNN
-F 2 "Resistor_SMD:R_0805_2012Metric_Pad1.15x1.40mm_HandSolder" H 5850 7100 50  0001 C CNN
+F 2 "Resistor_SMD:R_0805_2012Metric" H 5850 7100 50  0001 C CNN
 F 3 "~" H 5850 7100 50  0001 C CNN
 F 4 "C17673" H 5850 7100 50  0001 C CNN "LCSC#"
@@
 F 0 "R5" H 3759 3446 50  0000 L CNN
 F 1 "470" H 3759 3355 50  0000 L CNN
-F 2 "Resistor_SMD:R_0805_2012Metric_Pad1.15x1.40mm_HandSolder" H 3700 3400 50  0001 C CNN
+F 2 "Resistor_SMD:R_0805_2012Metric" H 3700 3400 50  0001 C CNN
 F 3 "~" H 3700 3400 50  0001 C CNN
 F 4 "C17710" H 3700 3400 50  0001 C CNN "LCSC#"

Commit message: Changed fuse to updated SMT part #
Parts:
- F1: LCSC# C151162 -> C70076
Changed lines of the file:
@@
 F 2 "Fuse:Fuse_1206_3216Metric" H 2400 2000 50  0001 L CNN
 F 3 "~" H 2350 2200 50  0001 C CNN
-F 4 "C151162" V 2350 2200 50  0001 C CNN "LCSC#"
+F 4 "C70076" V 2350 2200 50  0001 C CNN "LCSC#"
 	1    2350 2200
 	0    1    1    0

Commit message: Refilled zones, re-checked DRC
Connections:
- no-connect marks 2 -> 4
Changed lines of the file:
@@
 $EndComp
 Wire Wire Line
-	5000 5500 5250 5500
+	5000 5500 5200 5500
 $Comp
 L power:+5V #PWR0103
@@
 	1500 2200 2050 2200
 Wire Wire Line
-	1650 4600 1800 4600
-Wire Wire Line
 	7000 5500 7250 5500
 Wire Wire Line
@@
 	0    -1   -1   0
 $EndComp
+NoConn ~ 4500 5900
+NoConn ~ 5500 6100
+Connection ~ 2800 2200
+Wire Wire Line
+	5200 5500 5250 5500
+Wire Wire Line
+	1650 4600 1800 4600
 $EndSCHEMATC

Commit message: initial branch commit * very dirty - lots of overlapping traces * removed MOSFET * replaced diode footprints * WIP commit for remote storage
Parts:
- removed Q1: 2N7002, Package_TO_SOT_SMD:SOT-23, symbol Transistor_FET:2N7002
- removed R4: 4.7k, Resistor_SMD:R_0805_2012Metric, symbol Device:R_Small
- D1, D10, D11, D12, D13, D14, D15, D16, D17, D18, D19, D2, D20, D21, D22, D23, D24, D25, D26, D27, D28, D29, D3, D30, D31, D32, D33, D34, D35, D36, D37, D38, D39, D4, D40, D41, D42, D43, D44, D45, D46, D47, D48, D49, D5, D50, D51, D52, D53, D54, D55, D56, D57, D58, D59, D6, D60, D61, D62, D63, D64, D65, D66, D67, D68, D69, D7, D70, D71, D72, D73, D74, D75, D76, D77, D78, D79, D8, D80, D81, D82, D83, D84, D85, D9: footprint bear_face_parts:Diode-Hybrid-Back -> Diode_SMD:D_0805_2012Metric_Pad1.15x1.40mm_HandSolder
- J1: symbol Connector:USB_B_Micro -> bear_face_pcb-rescue:USB_B_Micro-Connector
- U1: symbol MCU_Microchip_ATmega:ATmega32U4-AU -> bear_face_pcb-rescue:ATmega32U4-AU-MCU_Microchip_ATmega
Connections:
- net LEDOUT is gone; now on net LEDPIN: R5.2
- net +5V: no longer U2.5 (VP)
- net DA+: no longer U2.4 (IO3)
- net DA-: no longer U2.3 (IO2)
- net GND: no longer U2.2 (VN)
Other:
- moved on the sheet: U2
