File: bear_face_pcb.sch (KiCad schematic (older format))
At the start: 199 parts, among them J1 USB_B_Micro-Connector, J2 Conn_02x03_Odd_Even, SW1 RESET, U1 ATmega32U4-AU, U2 SRV05-4, Y1 16MHz

Commit message: changed USB footprint
Parts:
- J1: footprint Connector_USB:USB_Micro-B_Wuerth_629105150521 -> bear_face_parts:MINI-USB-SMD_MICRO-4P-DIP
Changed lines of the file:
@@
 F 0 "J1" H 1057 2717 50  0000 C CNN
 F 1 "USB_B_Micro-Connector" H 1057 2626 50  0000 C CNN
-F 2 "Connector_USB:USB_Micro-B_Wuerth_629105150521" H 1150 2200 50  0001 C CNN
+F 2 "bear_face_parts:MINI-USB-SMD_MICRO-4P-DIP" H 1150 2200 50  0001 C CNN
 F 3 "" H 1150 2200 50  0001 C CNN
 F 4 "" H 1000 2250 50  0001 C CNN "LCSC"

Commit message: added symbol for graphics
Parts:
- G1, G2: symbol keebio:Hole -> bear_face_pcb:Graphic
- J1: LCSC (none) -> C456008
Other:
- moved on the sheet: H2, H3, H4, H6, H7, H8
Changed lines of the file:
@@
 L keebio:Hole H2
 U 1 1 5E007407
-P 1200 700
-F 0 "H2" H 1386 753 60  0000 L CNN
-F 1 "Hole" H 1386 647 60  0000 L CNN
-F 2 "bear_face_parts:MountingHole_6mm" H 1200 700 60  0001 C CNN
-F 3 "" H 1200 700 60  0001 C CNN
-	1    1200 700
+P 1300 700
+F 0 "H2" H 1486 753 60  0000 L CNN
+F 1 "Hole" H 1486 647 60  0000 L CNN
+F 2 "bear_face_parts:MountingHole_6mm" H 1300 700 60  0001 C CNN
+F 3 "" H 1300 700 60  0001 C CNN
+	1    1300 700
 	1    0    0    -1
 $EndComp
@@
 L keebio:Hole H3
 U 1 1 5E00740D
-P 1700 700
-F 0 "H3" H 1886 753 60  0000 L CNN
-F 1 "Hole" H 1886 647 60  0000 L CNN
-F 2 "bear_face_parts:MountingHole_6mm" H 1700 700 60  0001 C CNN
-F 3 "" H 1700 700 60  0001 C CNN
-	1    1700 700
+P 1900 700
+F 0 "H3" H 2086 753 60  0000 L CNN
+F 1 "Hole" H 2086 647 60  0000 L CNN
+F 2 "bear_face_parts:MountingHole_6mm" H 1900 700 60  0001 C CNN
+F 3 "" H 1900 700 60  0001 C CNN
+	1    1900 700
 	1    0    0    -1
 $EndComp
@@
 L keebio:Hole H7
 U 1 1 5E01E2A7
-P 1700 1200
-F 0 "H7" H 1886 1253 60  0000 L CNN
-F 1 "Hole" H 1886 1147 60  0000 L CNN
-F 2 "bear_face_parts:MountingHole_6mm" H 1700 1200 60  0001 C CNN
-F 3 "" H 1700 1200 60  0001 C CNN
-	1    1700 1200
+P 1900 1200
+F 0 "H7" H 2086 1253 60  0000 L CNN
+F 1 "Hole" H 2086 1147 60  0000 L CNN
+F 2 "bear_face_parts:MountingHole_6mm" H 1900 1200 60  0001 C CNN
+F 3 "" H 1900 1200 60  0001 C CNN
+	1    1900 1200
 	1    0    0    -1
 $EndComp
@@
 L keebio:Hole H6
 U 1 1 5E04EBAD
-P 1200 1200
-F 0 "H6" H 1386 1253 60  0000 L CNN
-F 1 "Hole" H 1386 1147 60  0000 L CNN
-F 2 "bear_face_parts:MountingHole_6mm" H 1200 1200 60  0001 C CNN
-F 3 "" H 1200 1200 60  0001 C CNN
-	1    1200 1200
+P 1300 1200
+F 0 "H6" H 1486 1253 60  0000 L CNN
+F 1 "Hole" H 1486 1147 60  0000 L CNN
+F 2 "bear_face_parts:MountingHole_6mm" H 1300 1200 60  0001 C CNN
+F 3 "" H 1300 1200 60  0001 C CNN
+	1    1300 1200
 	1    0    0    -1
 $EndComp
@@
 L keebio:Hole H4
 U 1 1 5E04EBB9
-P 2200 700
-F 0 "H4" H 2386 753 60  0000 L CNN
-F 1 "Hole" H 2386 647 60  0000 L CNN
-F 2 "bear_face_parts:MountingHole_6mm" H 2200 700 60  0001 C CNN
-F 3 "" H 2200 700 60  0001 C CNN
-	1    2200 700
+P 2500 700
+F 0 "H4" H 2686 753 60  0000 L CNN
+F 1 "Hole" H 2686 647 60  0000 L CNN
+F 2 "bear_face_parts:MountingHole_6mm" H 2500 700 60  0001 C CNN
+F 3 "" H 2500 700 60  0001 C CNN
+	1    2500 700
 	1    0    0    -1
 $EndComp
@@
 Connection ~ 5350 1750
 $Comp
-L keebio:Hole G1
-U 1 1 5E310D8F
-P 9500 5500
-F 0 "G1" H 9686 5553 60  0000 L CNN
-F 1 "FACE" H 9686 5447 60  0000 L CNN
-F 2 "bear_face_silks:cbf_small_flipped" H 9500 5500 60  0001 C CNN
-F 3 "" H 9500 5500 60  0001 C CNN
-	1    9500 5500
-	1    0    0    -1
-$EndComp
-$Comp
-L keebio:Hole G2
+L bear_face_pcb:Graphic G2
 U 1 1 5E3129DC
 P 10100 5500
@@
 L Connector_Generic:Conn_01x01 H8
 U 1 1 664A148D
-P 2200 1150
-F 0 "H8" H 1850 1100 50  0000 C CNN
-F 1 "Hole" H 1850 1200 50  0000 C CNN
-F 2 "bear_face_parts:MountingHole_3mm" H 2200 1150 50  0001 C CNN
-F 3 "~" H 2200 1150 50  0001 C CNN
-	1    2200 1150
+P 2500 1150
+F 0 "H8" H 2150 1100 50  0000 C CNN
+F 1 "Hole" H 2150 1200 50  0000 C CNN
+F 2 "bear_face_parts:MountingHole_3mm" H 2500 1150 50  0001 C CNN
+F 3 "~" H 2500 1150 50  0001 C CNN
+	1    2500 1150
 	-1   0    0    1
 $EndComp
@@
 L power:GND #PWR0111
 U 1 1 664D0BC7
-P 2400 1150
-F 0 "#PWR0111" H 2400 900 50  0001 C CNN
-F 1 "GND" H 2405 977 50  0000 C CNN
-F 2 "" H 2400 1150 50  0001 C CNN
-F 3 "" H 2400 1150 50  0001 C CNN
-	1    2400 1150
+P 2700 1150
+F 0 "#PWR0111" H 2700 900 50  0001 C CNN
+F 1 "GND" H 2705 977 50  0000 C CNN
+F 2 "" H 2700 1150 50  0001 C CNN
+F 3 "" H 2700 1150 50  0001 C CNN
+	1    2700 1150
 	1    0    0    -1
 $EndComp
@@
 F 2 "bear_face_parts:MINI-USB-SMD_MICRO-4P-DIP" H 1150 2200 50  0001 C CNN
 F 3 "" H 1150 2200 50  0001 C CNN
-F 4 "" H 1000 2250 50  0001 C CNN "LCSC"
+F 4 "C456008" H 1000 2250 50  0001 C CNN "LCSC"
 	1    1000 2250
 	1    0    0    -1
@@
 Wire Wire Line
 	1900 2250 2100 2250
+$Comp
+L bear_face_pcb:Graphic G1
+U 1 1 5E310D8F
+P 9500 5500
+F 0 "G1" H 9686 5553 60  0000 L CNN
+F 1 "FACE" H 9686 5447 60  0000 L CNN
+F 2 "bear_face_silks:cbf_small_flipped" H 9500 5500 60  0001 C CNN
+F 3 "" H 9500 5500 60  0001 C CNN
+	1    9500 5500
+	1    0    0    -1
+$EndComp
 $EndSCHEMATC

Commit message: inital stab placement * deleted no stab footprints * updated footprints for readability
Parts:
- MX29: footprint bear_face_parts:MXOnly-2U-NoLED-NoStabs -> bear_face_parts:MXOnly-2U-NoLED
- MX79: footprint bear_face_parts:MXOnly-6.25U-NoLED-NoStabs -> bear_face_parts:MXOnly-6.25U-ReversedStabilizers-NoLED
Changed lines of the file:
@@
 F 0 "MX79" H 6233 4823 60  0000 C CNN
 F 1 "SPACE" H 6233 4749 20  0000 C CNN
-F 2 "bear_face_parts:MXOnly-6.25U-NoLED-NoStabs" H 5575 4575 60  0001 C CNN
+F 2 "bear_face_parts:MXOnly-6.25U-ReversedStabilizers-NoLED" H 5575 4575 60  0001 C CNN
 F 3 "" H 5575 4575 60  0001 C CNN
 	1    6200 4600
@@
 F 0 "MX29" H 10233 2023 60  0000 C CNN
 F 1 "BKSPC" H 10233 1949 20  0000 C CNN
-F 2 "bear_face_parts:MXOnly-2U-NoLED-NoStabs" H 9575 1775 60  0001 C CNN
+F 2 "bear_face_parts:MXOnly-2U-NoLED" H 9575 1775 60  0001 C CNN
 F 3 "" H 9575 1775 60  0001 C CNN
 	1    10200 1800

Commit message: reversed ISO enter stabs
Parts:
- MX59: footprint bear_face_parts:MXOnly-ISO-ANSI-Enter -> bear_face_parts:MXOnly-ISO-ANSI-Enter-ReversedStabilizers
Changed lines of the file:
@@
 F 0 "MX59" H 10233 3423 60  0000 C CNN
 F 1 "ENTER" H 10233 3349 20  0000 C CNN
-F 2 "bear_face_parts:MXOnly-ISO-ANSI-Enter" H 9575 3175 60  0001 C CNN
+F 2 "bear_face_parts:MXOnly-ISO-ANSI-Enter-ReversedStabilizers" H 9575 3175 60  0001 C CNN
 F 3 "" H 9575 3175 60  0001 C CNN
 	1    10200 3200

Commit message: rotated ISO enter 90 degrees * fixed routing, GND fill
Parts:
- MX59: footprint bear_face_parts:MXOnly-ISO-ANSI-Enter-ReversedStabilizers -> bear_face_parts:MXOnly-ISO-ANSI-Enter-ReversedStabilizers-ROTATED
Changed lines of the file:
@@
 F 0 "MX59" H 10233 3423 60  0000 C CNN
 F 1 "ENTER" H 10233 3349 20  0000 C CNN
-F 2 "bear_face_parts:MXOnly-ISO-ANSI-Enter-ReversedStabilizers" H 9575 3175 60  0001 C CNN
+F 2 "bear_face_parts:MXOnly-ISO-ANSI-Enter-ReversedStabilizers-ROTATED" H 9575 3175 60  0001 C CNN
 F 3 "" H 9575 3175 60  0001 C CNN
 	1    10200 3200

Commit message: silks pullup to v3c
Parts:
- MX59: footprint bear_face_parts:MXOnly-ISO-ANSI-Enter-ReversedStabilizers-ROTATED -> bear_face_parts:MXOnly-ISO-ANSI-Enter-ReversedStabilizers
- SW1: footprint bear_face_parts:PushButton_6x6mm_TH_Pretty -> bear_face_parts:6x6mm_RESET
Changed lines of the file:
@@
 F 0 "MX59" H 10233 3423 60  0000 C CNN
 F 1 "ENTER" H 10233 3349 20  0000 C CNN
-F 2 "bear_face_parts:MXOnly-ISO-ANSI-Enter-ReversedStabilizers-ROTATED" H 9575 3175 60  0001 C CNN
+F 2 "bear_face_parts:MXOnly-ISO-ANSI-Enter-ReversedStabilizers" H 9575 3175 60  0001 C CNN
 F 3 "" H 9575 3175 60  0001 C CNN
 	1    10200 3200
@@
 F 0 "SW1" H 8200 6385 50  0000 C CNN
 F 1 "RESET" H 8200 6294 50  0000 C CNN
-F 2 "bear_face_parts:PushButton_6x6mm_TH_Pretty" H 8200 6300 50  0001 C CNN
+F 2 "bear_face_parts:6x6mm_RESET" H 8200 6300 50  0001 C CNN
 F 3 "~" H 8200 6300 50  0001 C CNN
 	1    8200 6100

Commit message: renumbered Resistors
Parts:
- renumbered H8 to H5, H5 to H6, H6 to H7, H7 to H8, R5 to R3, R6 to R4, R7 to R5
Changed lines of the file:
@@
 $EndComp
 $Comp
-L keebio:Hole H7
+L keebio:Hole H8
 U 1 1 5E01E2A7
 P 1900 1200
-F 0 "H7" H 2086 1253 60  0000 L CNN
+F 0 "H8" H 2086 1253 60  0000 L CNN
 F 1 "Hole" H 2086 1147 60  0000 L CNN
 F 2 "bear_face_parts:MountingHole_6mm" H 1900 1200 60  0001 C CNN
@@
 $EndComp
 $Comp
-L keebio:Hole H5
+L keebio:Hole H6
 U 1 1 5E04EBA7
 P 700 1200
-F 0 "H5" H 886 1253 60  0000 L CNN
+F 0 "H6" H 886 1253 60  0000 L CNN
 F 1 "Hole" H 886 1147 60  0000 L CNN
 F 2 "bear_face_parts:MountingHole_6mm" H 700 1200 60  0001 C CNN
@@
 $EndComp
 $Comp
-L keebio:Hole H6
+L keebio:Hole H7
 U 1 1 5E04EBAD
 P 1300 1200
-F 0 "H6" H 1486 1253 60  0000 L CNN
+F 0 "H7" H 1486 1253 60  0000 L CNN
 F 1 "Hole" H 1486 1147 60  0000 L CNN
 F 2 "bear_face_parts:MountingHole_6mm" H 1300 1200 60  0001 C CNN
@@
 $EndComp
 $Comp
-L power:GND #PWR015
+L power:GND #PWR019
 U 1 1 5E26A195
 P 1950 7450
-F 0 "#PWR015" H 1950 7200 50  0001 C CNN
+F 0 "#PWR019" H 1950 7200 50  0001 C CNN
 F 1 "GND" H 1955 7277 50  0000 C CNN
 F 2 "" H 1950 7450 50  0001 C CNN
@@
 $EndComp
 $Comp
-L power:GND #PWR011
+L power:GND #PWR015
 U 1 1 5E2B8FB1
 P 3850 6250
-F 0 "#PWR011" H 3850 6000 50  0001 C CNN
+F 0 "#PWR015" H 3850 6000 50  0001 C CNN
 F 1 "GND" H 3855 6077 50  0000 C CNN
 F 2 "" H 3850 6250 50  0001 C CNN
@@
 	1400 5450 1750 5450
 $Comp
-L power:GND #PWR010
+L power:GND #PWR013
 U 1 1 5E398B8C
 P 1400 5750
-F 0 "#PWR010" H 1400 5500 50  0001 C CNN
+F 0 "#PWR013" H 1400 5500 50  0001 C CNN
 F 1 "GND" H 1405 5577 50  0000 C CNN
 F 2 "" H 1400 5750 50  0001 C CNN
@@
 	4400 7300 4200 7300
 $Comp
-L power:+5V #PWR014
+L power:+5V #PWR017
 U 1 1 5E4623DC
 P 4200 7000
-F 0 "#PWR014" H 4200 6850 50  0001 C CNN
+F 0 "#PWR017" H 4200 6850 50  0001 C CNN
 F 1 "+5V" H 4215 7173 50  0000 C CNN
 F 2 "" H 4200 7000 50  0001 C CNN
@@
 	4200 7100 4400 7100
 $Comp
-L power:GND #PWR016
+L power:GND #PWR018
 U 1 1 5E47D9BC
 P 4200 7400
-F 0 "#PWR016" H 4200 7150 50  0001 C CNN
+F 0 "#PWR018" H 4200 7150 50  0001 C CNN
 F 1 "GND" H 4205 7227 50  0000 C CNN
 F 2 "" H 4200 7400 50  0001 C CNN
@@
 	4200 7300 4000 7300
 $Comp
-L power:+5V #PWR09
+L power:+5V #PWR08
 U 1 1 5E4994F7
 P 1600 4950
-F 0 "#PWR09" H 1600 4800 50  0001 C CNN
+F 0 "#PWR08" H 1600 4800 50  0001 C CNN
 F 1 "+5V" H 1615 5123 50  0000 C CNN
 F 2 "" H 1600 4950 50  0001 C CNN
@@
 Connection ~ 700  4650
 $Comp
-L power:GND #PWR08
+L power:GND #PWR07
 U 1 1 5E616792
 P 700 4800
-F 0 "#PWR08" H 700 4550 50  0001 C CNN
+F 0 "#PWR07" H 700 4550 50  0001 C CNN
 F 1 "GND" H 705 4627 50  0000 C CNN
 F 2 "" H 700 4800 50  0001 C CNN
@@
 	8400 6100 8500 6100
 $Comp
-L power:GND #PWR07
+L power:GND #PWR014
 U 1 1 5E709B12
 P 7850 6000
-F 0 "#PWR07" H 7850 5750 50  0001 C CNN
+F 0 "#PWR014" H 7850 5750 50  0001 C CNN
 F 1 "GND" H 7855 5827 50  0000 C CNN
 F 2 "" H 7850 6000 50  0001 C CNN
@@
 	8500 6100 8600 6100
 $Comp
-L power:+5V #PWR05
+L power:+5V #PWR011
 U 1 1 5E749519
 P 8500 5550
-F 0 "#PWR05" H 8500 5400 50  0001 C CNN
+F 0 "#PWR011" H 8500 5400 50  0001 C CNN
 F 1 "+5V" H 8515 5723 50  0000 C CNN
 F 2 "" H 8500 5550 50  0001 C CNN
@@
 	8500 5550 8500 5650
 $Comp
-L Device:R_Small R7
+L Device:R_Small R5
 U 1 1 5E285AAF
 P 3400 6250
-F 0 "R7" V 3204 6250 50  0000 C CNN
+F 0 "R5" V 3204 6250 50  0000 C CNN
 F 1 "10k" V 3295 6250 50  0000 C CNN
 F 2 "Resistor_SMD:R_0805_2012Metric" H 3400 6250 50  0001 C CNN
@@
 	1100 4650 1100 4750
 $Comp
-L power:+5V #PWR0103
+L power:+5V #PWR09
 U 1 1 5E32F6EA
 P 5250 5500
-F 0 "#PWR0103" H 5250 5350 50  0001 C CNN
+F 0 "#PWR09" H 5250 5350 50  0001 C CNN
 F 1 "+5V" H 5265 5673 50  0000 C CNN
 F 2 "" H 5250 5500 50  0001 C CNN
@@
 $EndComp
 $Comp
-L power:GND #PWR0104
+L power:GND #PWR016
 U 1 1 5E3845E4
 P 5000 6550
-F 0 "#PWR0104" H 5000 6300 50  0001 C CNN
+F 0 "#PWR016" H 5000 6300 50  0001 C CNN
 F 1 "GND" H 5005 6377 50  0000 C CNN
 F 2 "" H 5000 6550 50  0001 C CNN
@@
 RESET
 $Comp
-L power:GND #PWR0105
+L power:GND #PWR012
 U 1 1 5E4F520E
 P 7250 5700
-F 0 "#PWR0105" H 7250 5450 50  0001 C CNN
+F 0 "#PWR012" H 7250 5450 50  0001 C CNN
 F 1 "GND" H 7255 5527 50  0000 C CNN
 F 2 "" H 7250 5700 50  0001 C CNN
@@
 $EndComp
 $Comp
-L power:+5V #PWR0106
+L power:+5V #PWR010
 U 1 1 5E54EE72
 P 7250 5500
-F 0 "#PWR0106" H 7250 5350 50  0001 C CNN
+F 0 "#PWR010" H 7250 5350 50  0001 C CNN
 F 1 "+5V" H 7265 5673 50  0000 C CNN
 F 2 "" H 7250 5500 50  0001 C CNN
@@
 DB+
 $Comp
-L Connector_Generic:Conn_01x01 H8
+L Connector_Generic:Conn_01x01 H5
 U 1 1 664A148D
 P 2500 1150
-F 0 "H8" H 2150 1100 50  0000 C CNN
+F 0 "H5" H 2150 1100 50  0000 C CNN
 F 1 "Hole" H 2150 1200 50  0000 C CNN
 F 2 "bear_face_parts:MountingHole_3mm" H 2500 1150 50  0001 C CNN
@@
 $EndComp
 $Comp
-L power:GND #PWR0111
+L power:GND #PWR01
 U 1 1 664D0BC7
 P 2700 1150
-F 0 "#PWR0111" H 2700 900 50  0001 C CNN
+F 0 "#PWR01" H 2700 900 50  0001 C CNN
 F 1 "GND" H 2705 977 50  0000 C CNN
 F 2 "" H 2700 1150 50  0001 C CNN
@@
 	3700 3500 3300 3500
 $Comp
-L power:+5V #PWR0107
+L power:+5V #PWR05
 U 1 1 5E6EBC56
 P 3400 3200
-F 0 "#PWR0107" H 3400 3050 50  0001 C CNN
+F 0 "#PWR05" H 3400 3050 50  0001 C CNN
 F 1 "+5V" H 3415 3373 50  0000 C CNN
 F 2 "" H 3400 3200 50  0001 C CNN
@@
 $EndComp
 $Comp
-L Device:R_Small R6
+L Device:R_Small R4
 U 1 1 5E729BAE
 P 8500 5750
-F 0 "R6" H 8559 5796 50  0000 L CNN
+F 0 "R4" H 8559 5796 50  0000 L CNN
 F 1 "10k" H 8559 5705 50  0000 L CNN
 F 2 "Resistor_SMD:R_0805_2012Metric" H 8500 5750 50  0001 C CNN
@@
 $EndComp
 $Comp
-L Device:R_Small R5
+L Device:R_Small R3
 U 1 1 5E6C94F1
 P 3700 3400
-F 0 "R5" H 3759 3446 50  0000 L CNN
+F 0 "R3" H 3759 3446 50  0000 L CNN
 F 1 "470" H 3759 3355 50  0000 L CNN
 F 2 "Resistor_SMD:R_0805_2012Metric" H 3700 3400 50  0001 C CNN
@@
 	1000 2650 1150 2650
 $Comp
-L power:GND #PWR0101
+L power:GND #PWR04
 U 1 1 6578DF34
 P 1150 2650
-F 0 "#PWR0101" H 1150 2400 50  0001 C CNN
+F 0 "#PWR04" H 1150 2400 50  0001 C CNN
 F 1 "GND" H 1155 2477 50  0000 C CNN
 F 2 "" H 1150 2650 50  0001 C CNN

Commit message: final silks tweaks, final gerbers
Parts:
- MX27: value (_-) -> -_
- MX28: value (+) -> =+
- MX42: value [ -> [{
- MX43: value ] -> ]}
Changed lines of the file:
@@
 P 9700 2500
 F 0 "MX43" H 9733 2723 60  0000 C CNN
-F 1 "]" H 9733 2649 20  0000 C CNN
+F 1 "]}" H 9733 2649 20  0000 C CNN
 F 2 "bear_face_parts:MXOnly-1U-NoLED" H 9075 2475 60  0001 C CNN
 F 3 "" H 9075 2475 60  0001 C CNN
@@
 P 9200 2500
 F 0 "MX42" H 9233 2723 60  0000 C CNN
-F 1 "[" H 9233 2649 20  0000 C CNN
+F 1 "[{" H 9233 2649 20  0000 C CNN
 F 2 "bear_face_parts:MXOnly-1U-NoLED" H 8575 2475 60  0001 C CNN
 F 3 "" H 8575 2475 60  0001 C CNN
@@
 P 9700 1800
 F 0 "MX28" H 9733 2023 60  0000 C CNN
-F 1 "(+)" H 9733 1949 20  0000 C CNN
+F 1 "=+" H 9733 1949 20  0000 C CNN
 F 2 "bear_face_parts:MXOnly-1U-NoLED" H 9075 1775 60  0001 C CNN
 F 3 "" H 9075 1775 60  0001 C CNN
@@
 P 9200 1800
 F 0 "MX27" H 9233 2023 60  0000 C CNN
-F 1 "(_-)" H 9233 1949 20  0000 C CNN
+F 1 "-_" H 9233 1949 20  0000 C CNN
 F 2 "bear_face_parts:MXOnly-1U-NoLED" H 8575 1775 60  0001 C CNN
 F 3 "" H 8575 1775 60  0001 C CNN
