File: bear_face_pcb.kicad_sch (KiCad schematic)
At the start: 199 parts, among them J1 USB_B_Micro-Connector, J2 Conn_02x03_Odd_Even, SW1 RESET, U1 ATmega32U4-AU, U2 SRV05-4, Y1 16MHz

Commit message: plate ground, fmask changes * still need to round corners * need new gerbers
Parts:
- H5: footprint MountingHole:MountingHole_2.2mm_M2_Pad -> bear_face_parts:MountingHole_Header_Pin_Pad
Changed lines of the file:
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@@
       (effects (font (size 1.27 1.27)))
     )
-    (property "Footprint" "MountingHole:MountingHole_2.2mm_M2_Pad" (at 63.5 29.21 0)
+    (property "Footprint" "bear_face_parts:MountingHole_Header_Pin_Pad" (at 63.5 29.21 0)
       (effects (font (size 1.27 1.27)) hide)
     )

Commit message: repo cleanup in favor of JLC plugin
Parts:
- H10, H3, H4, H5, H6, H7, H8, H9, SW1: now not fitted
Changed lines of the file:
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@@
   )
   (symbol (lib_id "Switch:SW_Push") (at 208.28 154.94 0) (unit 1)
-    (in_bom yes) (on_board yes) (dnp no)
+    (in_bom yes) (on_board yes) (dnp yes)
     (property "Reference" "SW1" (at 208.28 147.701 0)
       (effects (font (size 1.27 1.27)))
@@
   )
   (symbol (lib_id "keebio:Hole") (at 33.02 17.78 0) (unit 1)
-    (in_bom yes) (on_board yes) (dnp no)
+    (in_bom yes) (on_board yes) (dnp yes)
     (property "Reference" "H7" (at 37.7444 16.4338 0)
       (effects (font (size 1.524 1.524)) (justify left))
@@
   )
   (symbol (lib_id "keebio:Hole") (at 48.26 17.78 0) (unit 1)
-    (in_bom yes) (on_board yes) (dnp no)
+    (in_bom yes) (on_board yes) (dnp yes)
     (property "Reference" "H8" (at 52.9844 16.4338 0)
       (effects (font (size 1.524 1.524)) (justify left))
@@
   )
   (symbol (lib_id "keebio:Hole") (at 48.26 30.48 0) (unit 1)
-    (in_bom yes) (on_board yes) (dnp no)
+    (in_bom yes) (on_board yes) (dnp yes)
     (property "Reference" "H9" (at 52.9844 29.1338 0)
       (effects (font (size 1.524 1.524)) (justify left))
@@
   )
   (symbol (lib_id "keebio:Hole") (at 17.78 17.78 0) (unit 1)
-    (in_bom yes) (on_board yes) (dnp no)
+    (in_bom yes) (on_board yes) (dnp yes)
     (property "Reference" "H4" (at 22.5044 16.4338 0)
       (effects (font (size 1.524 1.524)) (justify left))
@@
   )
   (symbol (lib_id "keebio:Hole") (at 17.78 30.48 0) (unit 1)
-    (in_bom yes) (on_board yes) (dnp no)
+    (in_bom yes) (on_board yes) (dnp yes)
     (property "Reference" "H3" (at 22.5044 29.1338 0)
       (effects (font (size 1.524 1.524)) (justify left))
@@
   )
   (symbol (lib_id "keebio:Hole") (at 33.02 30.48 0) (unit 1)
-    (in_bom yes) (on_board yes) (dnp no)
+    (in_bom yes) (on_board yes) (dnp yes)
     (property "Reference" "H6" (at 37.7444 29.1338 0)
       (effects (font (size 1.524 1.524)) (justify left))
@@
   )
   (symbol (lib_id "keebio:Hole") (at 63.5 17.78 0) (unit 1)
-    (in_bom yes) (on_board yes) (dnp no)
+    (in_bom yes) (on_board yes) (dnp yes)
     (property "Reference" "H10" (at 68.2244 16.4338 0)
       (effects (font (size 1.524 1.524)) (justify left))
@@
   )
   (symbol (lib_id "Connector_Generic:Conn_01x01") (at 63.5 29.21 180) (unit 1)
-    (in_bom yes) (on_board yes) (dnp no)
+    (in_bom yes) (on_board yes) (dnp yes)
     (property "Reference" "H5" (at 72.39 27.94 0)
       (effects (font (size 1.27 1.27)))
