File: bear_face_pcb.kicad_pcb (KiCad board)
At the start: 2 copper layers, 300 x 112.2 mm, 216 parts, among them J1 USB-C, J2 Conn_02x03_Odd_Even, SW1 RESET, U1 ATmega32U4-AU, U2 SRV05-4, Y1 16MHz

Commit message: rounded stab area pcb, new gerbers, minor silks tweaks
Parts:
- Hc10, Hc3, Hc4, Hc8: footprint bear_face_parts:MountingHole_6mm -> MountingHole:MountingHole_2.2mm_M2_Pad
- moved D85 11.1 mm to (343.7, 176.3)
- moved Hc4 0.27 mm to (84.1, 118.8)
- moved Hc10 0.17 mm to (105.5, 171.6)
Routing:
- net ROW5: track 309.5 -> 298.6 mm
- net Net-(D85-A): track 9.47 -> 19.2 mm
- net COL7: track 154.8 -> 154.1 mm
- net GND: vias 17 -> 16
Other:
- outline, holes or cut-outs redrawn

Commit message: cleaned up edge cuts, new gerbers
Changed lines of the file:
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@@
   (gr_line (start 79.68 68.834) (end 88.062 68.834)
     (stroke (width 0.15) (type dash)) (layer "Cmts.User"))
-  (gr_line (start 354.319106 70.059859) (end 66.312 70.060358)
+  (gr_line (start 354.319106 70.0604) (end 66.312 70.0604)
     (stroke (width 0.12) (type solid)) (layer "Edge.Cuts"))
   (gr_line (start 60.312 91.201) (end 60.312 121.226)
     (stroke (width 0.12) (type solid)) (layer "Edge.Cuts"))
-  (gr_line (start 360.312 79.651002) (end 360.308814 82.725999)
+  (gr_line (start 360.312 79.651002) (end 360.312 82.725999)
     (stroke (width 0.12) (type solid)) (layer "Edge.Cuts"))
   (gr_line (start 360.312 91.222777) (end 360.312 121.236)
@@
   (gr_arc (start 360.065012 90.975999) (mid 356.304383 86.977504) (end 360.06201 82.976188)
     (stroke (width 0.12) (type solid)) (layer "Edge.Cuts"))
-  (gr_arc (start 360.32 175.652072) (mid 358.821399 179.224449) (end 355.240091 180.701587)
-    (stroke (width 0.12) (type solid)) (layer "Edge.Cuts"))
-  (gr_line (start 236.832734 180.702734) (end 141.030366 180.702413)
+  (gr_line (start 236.832734 180.702413) (end 141.030366 180.702413)
     (stroke (width 0.12) (type default)) (layer "Edge.Cuts"))
-  (gr_arc (start 360.064933 167.559147) (mid 360.246694 167.634302) (end 360.322 167.816)
+  (gr_arc (start 360.064933 167.559147) (mid 360.241686 167.636381) (end 360.312 167.816)
     (stroke (width 0.12) (type default)) (layer "Edge.Cuts"))
   (gr_arc (start 60.312384 129.718716) (mid 60.376781 129.55067) (end 60.537 129.468716)
@@
   (gr_arc (start 360.064933 167.559146) (mid 356.320451 163.580833) (end 360.055286 159.593462)
     (stroke (width 0.12) (type solid)) (layer "Edge.Cuts"))
-  (gr_line (start 359.312 78.651002) (end 356.319106 78.65)
+  (gr_line (start 359.312 78.65) (end 356.319106 78.65)
     (stroke (width 0.12) (type default)) (layer "Edge.Cuts"))
-  (gr_arc (start 65.312 77.650499) (mid 65.019107 78.357606) (end 64.312 78.650499)
+  (gr_arc (start 65.312 77.65) (mid 65.01921 78.357356) (end 64.312 78.650499)
     (stroke (width 0.12) (type default)) (layer "Edge.Cuts"))
   (gr_arc (start 60.5634 140.4802) (mid 64.318695 144.478811) (end 60.563777 148.477776)
     (stroke (width 0.12) (type solid)) (layer "Edge.Cuts"))
-  (gr_arc (start 60.319106 79.651501) (mid 60.611999 78.944396) (end 61.319106 78.651501)
+  (gr_arc (start 60.319106 79.651002) (mid 60.611998 78.943895) (end 61.319106 78.651002)
     (stroke (width 0.12) (type default)) (layer "Edge.Cuts"))
-  (gr_arc (start 65.312 71.060358) (mid 65.604893 70.353251) (end 66.312 70.060358)
+  (gr_arc (start 65.312 71.060358) (mid 65.604908 70.353278) (end 66.312 70.0604)
     (stroke (width 0.12) (type default)) (layer "Edge.Cuts"))
-  (gr_arc (start 360.308814 82.725999) (mid 360.23673 82.901717) (end 360.06201 82.976188)
+  (gr_arc (start 360.312 82.725999) (mid 360.238322 82.90237) (end 360.06201 82.976188)
     (stroke (width 0.12) (type default)) (layer "Edge.Cuts"))
   (gr_arc (start 359.312 78.651002) (mid 360.019106 78.943895) (end 360.312 79.651002)
@@
   (gr_arc (start 60.562001 159.550999) (mid 60.385224 159.477776) (end 60.312001 159.300999)
     (stroke (width 0.12) (type default)) (layer "Edge.Cuts"))
-  (gr_line (start 64.312 78.650499) (end 61.319106 78.651501)
+  (gr_line (start 64.312 78.651501) (end 61.319106 78.651501)
     (stroke (width 0.12) (type default)) (layer "Edge.Cuts"))
   (gr_line (start 60.312 167.801) (end 60.312 175.622504)
@@
   (gr_line (start 60.319106 79.651501) (end 60.319106 82.749223)
     (stroke (width 0.12) (type default)) (layer "Edge.Cuts"))
-  (gr_line (start 360.322 167.816) (end 360.32 175.652072)
+  (gr_arc (start 360.311999 175.652072) (mid 358.816863 179.223117) (end 355.240095 180.70451)
+    (stroke (width 0.12) (type solid)) (layer "Edge.Cuts"))
+  (gr_line (start 360.312 167.816) (end 360.312 175.652072)
     (stroke (width 0.12) (type default)) (layer "Edge.Cuts"))
   (gr_line (start 60.313777 129.718716) (end 60.313777 140.224223)
     (stroke (width 0.12) (type default)) (layer "Edge.Cuts"))
-  (gr_line (start 355.240091 180.702413) (end 241.068266 180.702734)
+  (gr_line (start 355.240091 180.702413) (end 241.068266 180.702413)
     (stroke (width 0.12) (type default)) (layer "Edge.Cuts"))
   (gr_arc (start 141.030366 180.702413) (mid 138.9126 182.244679) (end 136.794834 180.702413)
