File: bear_face_pcb.kicad_pcb (KiCad board)
At the start: 2 copper layers, 300 x 112.2 mm, 216 parts, among them J1 USB-C, J2 Conn_02x03_Odd_Even, SW1 RESET, U1 ATmega32U4-AU, U2 SRV05-4, Y1 16MHz

Commit message: fixed spacebar stabilizer holes * bottom-edge stabilizer holes should not need to be filed down now * generated new gerbers (not tested)
Other:
- board size 300 x 112.2 mm -> 300 x 111.8 mm

Commit message: fixed silkscreen versioning, added new gerbers
Other:
- board text added: "bear_face v3.2c designed by /u/chemicalwill"
- board text removed: "bear_face v3.1c designed by /u/chemicalwill"
Changed lines of the file:
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@@
 		(layer "Edge.Cuts")
 	)
-	(gr_text "bear_face v3.1c\ndesigned by /u/chemicalwill"
+	(gr_text "bear_face v3.2c\ndesigned by /u/chemicalwill"
 		(at 218.312 170.688 0)
 		(layer "B.SilkS")
